File: kicad/audio.kicad_sch (KiCad schematic)
At the start: 29 parts, among them J3 DMA58-4 (4 ohm), Q4 AO3401A, U10 LTC4412ES6, U9 TAS5760M (DCA-48)

Commit message: schematic second pass
Parts:
- removed C163, C187: 100nF, Capacitor_SMD:C_0603_1608Metric, symbol Device:C
- U9: value TAS5760M (DCA-48) -> TAS5760MDAPR; footprint Package_SO:TSSOP-48_6.1x12.5mm_P0.5mm -> Package_SO:HTSSOP-32-1EP_6.1x11mm_P0.65mm_EP5.2x11mm_Mask4.11x4.36mm
Connections:
- net +3V3: now also U9.1 (AVDD), U9.10 (DVDD); no longer U9.46 (AVDD), U9.9 (DVDD)
- net AMP_ADR: now also U9.13 (SPK_SLEEP/ADR); no longer U9.12 (SPK_SLEEP/ADR)
- net AMP_ANAREF: now also U9.5 (ANA_REF); no longer U9.4 (ANA_REF)
- net AMP_ANAREG: now also U9.3 (ANA_REG); no longer U9.2 (ANA_REG)
- net AMP_BSTRPA+: now also U9.30 (BSTRPA+); no longer U9.43 (BSTRPA+)
- net AMP_BSTRPA-: now also U9.25 (BSTRPA-); no longer U9.39 (BSTRPA-)
- net AMP_BSTRPB+: now also U9.19 (BSTRPB+); no longer U9.34 (BSTRPB+)
- net AMP_BSTRPB-: now also U9.24 (BSTRPB-); no longer U9.38 (BSTRPB-)
- net AMP_GAIN: now also U9.12 (SPK_GAIN1); no longer U9.10 (SPK_GAIN0)
- net AMP_GVDD: now also U9.2 (SFT_CLIP), U9.32 (GVDD_REG); no longer U9.1 (SFT_CLIP), U9.48 (GVDD_REG)
- net AMP_OUTN: now also U9.23 (SPK_OUTB-), U9.26 (SPK_OUTA-); no longer U9.37 (SPK_OUTB-), U9.40 (SPK_OUTA-)
- net AMP_OUTP: now also U9.20 (SPK_OUTB+), U9.29 (SPK_OUTA+); no longer U9.35 (SPK_OUTB+), U9.42 (SPK_OUTA+)
- net AMP_VCOM: now also U9.4 (VCOM); no longer U9.3 (VCOM)
- net GND: now also C170.1, C171.1, C172.1, D30.1 (K), Q4.3 (D), U10.6 (SENSE), U9.33 (PAD); no longer U9.17 (DGND), U9.19 (NC), U9.20 (NC), U9.23 (NC), U9.24 (NC), U9.25 (NC), U9.26 (NC), U9.29 (NC), U9.30 (NC), U9.36 (PGND), U9.41 (PGND), U9.47 (GGND), U9.49 (PAD)
- net I2C_SCL: now also U9.9 (PBTL/SCL); no longer U9.8 (PBTL/SCL)
- net I2C_SDA: now also U9.8 (FREQ/SDA); no longer U9.7 (FREQ/SDA)
- net I2S_BCLK: now also U9.15 (SCLK); no longer U9.14 (SCLK)
- net I2S_DOUT: now also U9.16 (SDIN); no longer U9.15 (SDIN)
- net I2S_LRCLK: now also U9.17 (LRCK); no longer U9.16 (LRCK)
- net I2S_MCLK: now also U9.14 (MCLK); no longer U9.13 (MCLK)
- net SPK_FAULT: now also U9.6 (SPK_FAULT); no longer U9.5 (SPK_FAULT)
- net SPK_SD: now also U9.7 (SPK_SD); no longer U9.6 (SPK_SD)
- removed net PVDD: C170.1, C171.1, C172.1, D30.1 (K), Q4.3 (D), U10.6 (SENSE), U9.32 (PVDD), U9.33 (PVDD), U9.44 (PVDD), U9.45 (PVDD)
Other:
- note added: "AUDIO — TAS5760M (DAP-32) PBTL mono + LTC4412 PVDD mux (12V<->5V) + LC filter"
- note added: "Bootstrap caps 33nF: VERIFY vs TAS5760M datasheet. PVDD = 12V(plugged)/5V(batt)."
- note removed: "AUDIO — TAS5760M PBTL mono + LTC4412 PVDD mux (12V<->5V) + LC filter"
- note removed: "Bootstrap caps 33nF: VERIFY value vs TAS5760M datasheet."
- note removed: "PVDD = 12V (plugged, via Schottky) OR 5V (battery, via LTC4412 FET) -> quieter alarm."
