File: kicad/charger.kicad_sch (KiCad schematic)
At the start: 37 parts, among them Q1 2N7002, Q2 AO3401A, Q3 2N7002, U2 LT3652EMSE, U3 AP9101CK6-BX, U4 AOSD32334C

Commit message: schematic second pass
Connections:
- net CH_VM is gone; now on net CH_APVDD: R21.1, U3.2 (VM)
- net CH_DIVND: no longer names the net of Q3.3 (D), R23.2
- net CH_FETMID: no longer names the net of U4.5 (D1), U4.6 (D1), U4.7 (D2), U4.8 (D2)
- net CH_FULLND: no longer names the net of Q1.3 (D), R16.2
- net CH_NTC2: no longer names the net of R17.1, RT1.2
- net CH_SENSE: no longer names the net of R18.1, U2.10 (SENSE)
Other:
- note added: "Cell- path: BATT- -> AOSD32334C (DO/CO gated) -> TCO 77C -> GND (PACK-)."
- note added: "Vbat -> ADC IO1 (VBAT_SENSE); FULLCHG_EN=4.2V mode; VBAT_DIV_EN gates the divider."
- note removed: "NTC on the 18650 holder (0/45 C window)"
- note removed: "TCO one-shot thermal fuse in series with the cell -"
- note removed: "Vbat -> ADC IO1 (VBAT_SENSE); FET gate = VBAT_DIV_EN (off in deep-sleep)"
