File: kicad/rails.kicad_sch (KiCad schematic)
At the start: 32 parts, among them U5 TPS61023, U6 TLV62569DBVR, U7 TPS55340PWPR

Commit message: schematic second pass
Connections:
- net RAIL12_CC: no longer names the net of C134.1, R48.2
- net RAIL33_SW: no longer names the net of L3.1, U6.3 (SW)
Other:
- note added: "12 V boost PLUGGED-ONLY: firmware asserts BOOST12_EN only when PD_PG live."
- note removed: "12 V boost is PLUGGED-ONLY: firmware asserts BOOST12_EN only when PD_PG live."
