File: kicad/clock.kicad_sch (KiCad schematic)
At the start: 169 parts, among them J1 USB4105-GF-A, J2 PROG, J3 Speaker DMA58-4 (4R), J4 X40.879 stepper (1e-4e, 1i-4i), J5 LS032B7DD02 (FH34SRJ-10S), J6 DM3AT-SF-PEJM5, J7 Sensor board (BME688+TSL2591+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, J8 Panel LEDs 5V (CLM3C x12), J9 Wake COB 12V (warm+cool), Q1 2N7002, Q2 AO3401A, Q3 2N7002, Q4 AO3401A, Q5 AO3400A, Q6 AO3400A, Q7 AO3400A, SW1 RESET, SW2 BOOT, SW3 EC11 encoder, SW4 BTN1, SW5 BTN2, SW6 BTN3, U1 CH224K, U10 LTC4412ES6, U11 TB6612FNG, U12 TB6612FNG, U13 MCP23017, U14 QRE1113, U2 LT3652EMSE, U3 AP9101CK6-BX, U4 AOSD32334C, U5 TPS61023, U6 TLV62569DBVR, U7 TPS55340PWPR, U8 ESP32-S3-WROOM-1-N16R8, U9 TAS5760MDAPR, Y1 32.768kHz

Commit message: manual schematic modification
Connections:
- net +3V3: now also R62.1; no longer R62.2
- net SPK_FAULT: now also R62.2; no longer R62.1
Other:
- moved on the sheet: C1, C105, C110, C135, C144, C145, C146, C162, C164, C165, C166, C172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

Commit message: fix schematic
Parts:
- removed SW3: EC11 encoder, Rotary_Encoder:RotaryEncoder_Alps_EC11E-Switch_Vertical_H20mm, symbol Device:RotaryEncoder_Switch
- removed SW4: BTN1, Button_Switch_SMD:SW_SPST_CK_RS282G05A3, symbol Switch:SW_Push
- removed SW5: BTN2, Button_Switch_SMD:SW_SPST_CK_RS282G05A3, symbol Switch:SW_Push
- removed SW6: BTN3, Button_Switch_SMD:SW_SPST_CK_RS282G05A3, symbol Switch:SW_Push
- added J10: UI: EC11 + 3 buttons (off-board), Connector_JST:JST_SH_SM08B-SRSS-TB_1x08-1MP_P1.00mm_Horizontal, symbol Connector_Generic:Conn_01x08
- C180, C181, C182, C183: value 33nF -> 220nF
- F1: footprint (none) -> clock:Fuse_TCO_Cantherm_SDF_L10.5mm_D4.0mm_P20.32mm_Horizontal
- J5: footprint Connector_FFC-FPC:Hirose_FH12-10S-0.5SH_1x10-1MP_P0.50mm_Horizontal -> clock:Hirose_FH34SRJ-10S-0.5SH_1x10-1MP_P0.50mm_Horizontal
- U14: value QRE1113 -> QRE1113GR; footprint (none) -> clock:OnSemi_QRE1113GR
Connections:
- net GND: now also J10.1 (Pin_1), J10.8 (Pin_8)
- net at R100.2, U8.24 (IO47_ENC_A): now also J10.2 (Pin_2)
- net at R101.2, U8.25 (IO48_ENC_B): now also J10.3 (Pin_3)
- net at U13.27 (GPA6): now also J10.7 (Pin_7)
- net at U13.25 (GPA4): now also J10.5 (Pin_5)
- net at U13.24 (GPA3): now also J10.4 (Pin_4)
- net at U13.26 (GPA5): now also J10.6 (Pin_6)
Other:
- note added: "INT: any GPA/GPB change -> IO44 (IOCON.MIRROR=1). EC11 + buttons mount on the"
- note added: "QRE1113GR faces reflective tabs on the hand hubs (no magnets)."
- note added: "Switch lines: MCP internal pull-ups + IOC. Encoder A/B -> PCNT (IO47/48), R100/R101 PU."
- note added: "enclosure -> JST SH cable to J10 (1 GND, 2 ENC_A, 3 ENC_B, 4-6 BTN1-3, 7 ENC_SW, 8 GND)."
- note added: "strips, encoder+buttons, cell) enter via connectors J1..J10 / BT1."
- note removed: "INT: any GPA/GPB change -> IO44 (IOCON.MIRROR=1). Buttons/encoder-switch"
- note removed: "QRE1113 faces reflective tabs on the hand hubs (no magnets)."
- note removed: "strips, cell) enter through connectors J1..J9 / BT1."
- note removed: "use MCP internal pull-ups. Encoder A/B -> hardware PCNT (IO47/48)."

Commit message: improve schematic with custom layout
Parts:
- removed J4: X40.879 stepper (1e-4e, 1i-4i), Connector_JST:JST_PH_B8B-PH-K_1x08_P2.00mm_Vertical, symbol Connector_Generic:Conn_01x08
- removed U3: AP9101CK6-BX, Package_TO_SOT_SMD:SOT-23-6, symbol Battery_Management:AP9101CK6
- added M1: X40.879, clock:Juken_X40-879_DualShaft, symbol clock:X40_879
- added U3: HY2111-GB, Package_TO_SOT_SMD:SOT-23-6, symbol clock:HY2111
- R20: value 330R -> 100R
- R21: value 2.7k -> 2k
Connections:
- net at U11.1 (AO1), U11.2 (AO1): now also M1.1 (1e)
- net at U11.5 (AO2), U11.6 (AO2): now also M1.2 (2e)
- net at U11.7 (BO2), U11.8 (BO2): now also M1.3 (3e)
- net at U11.11 (BO1), U11.12 (BO1): now also M1.4 (4e)
- net at U12.1 (AO1), U12.2 (AO1): now also M1.5 (1i)
- net at U12.5 (AO2), U12.6 (AO2): now also M1.6 (2i)
- net at U12.7 (BO2), U12.8 (BO2): now also M1.7 (3i)
- net at U12.11 (BO1), U12.12 (BO1): now also M1.8 (4i)
- net at C109.1, R20.2: now also U3.5 (VDD)
- net at BT1.2 (Pin_2), C109.2, U4.3 (S1): now also U3.6 (VSS)
- net at U4.2 (G2): now also U3.3 (OC)
- net at U4.4 (G1): now also U3.1 (OD)
- net at R21.1: now also U3.2 (CS)
Other:
- note added: "OV 4.28 V / OD 2.90 V fixed (-GB). Independent of the charger."
- note added: "cell- -> AOSD32334C (OD/OC gated) -> TCO 77 C -> PACK- (GND)"
- note removed: "OV 4.28 V / OD 2.80 V fixed (-BX). Independent of the charger."
- note removed: "cell- -> AOSD32334C (DO/CO gated) -> TCO 77 C -> PACK- (GND)"
