File: kicad/clock.kicad_sch (KiCad schematic)
At the start: 166 parts, among them J1 USB4105-GF-A, J10 UI: EC11 + 3 buttons (off-boa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, J2 PROG, J3 Speaker DMA58-4 (4R), J5 LS032B7DD02 (FH34SRJ-10S), J6 DM3AT-SF-PEJM5, J7 Sensor board (BME688+TSL2591+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, J8 Panel LEDs 5V (CLM3C x12), J9 Wake COB 12V (warm+cool), M1 X40.879, Q1 2N7002, Q2 AO3401A, Q3 2N7002, Q4 AO3401A, Q5 AO3400A, Q6 AO3400A, Q7 AO3400A, SW1 RESET, SW2 BOOT, U1 CH224K, U10 LTC4412ES6, U11 TB6612FNG, U12 TB6612FNG, U13 MCP23017, U14 QRE1113GR, U2 LT3652EMSE, U3 HY2111-GB, U4 AOSD32334C, U5 TPS61023, U6 TLV62569DBVR, U7 TPS55340PWPR, U8 ESP32-S3-WROOM-1-N16R8, U9 TAS5760MDAPR, Y1 32.768kHz

Commit message: cube redesign (v0.19): rewrite spec, drop display from schematic + BOM
- README: walnut cube + aluminum face/knob form factor, single-knob UX,
  NeoPixel status/dial LEDs, vertical USB-C, R14 retired; BOM + decision log
- kicad: remove Sharp LS032B7DD02 + FH34 (J5), panel caps, LCD_DISP/LCD_CS;
  SPI2 now microSD-only (b_display.py -> b_sd.py); datasheet/ untouched

Co-Authored-By: Claude Fable 5 <noreply@anthropic.com>
Parts:
- removed C220, C221: 1uF, Capacitor_SMD:C_0603_1608Metric, symbol Device:C
- removed J5: LS032B7DD02 (FH34SRJ-10S), clock:Hirose_FH34SRJ-10S-0.5SH_1x10-1MP_P0.50mm_Horizontal, symbol Connector_Generic:Conn_01x10
Connections:
- net LCD_DISP: no longer names the net of U13.4 (GPB3)
- no-connect marks 16 -> 18
Other:
- note added: "Layout: C222/C223 at the J6 VDD pin."
- note added: "STORAGE — microSD (DM3AT), SPI2 dedicated"
- note removed: "DISPLAY (LS032B7DD02, FPC) + microSD — shared SPI2"
- note removed: "EXTMODE=L -> software VCOM (frame-inversion bit, >=1 Hz)."
- note removed: "Layout: C220/C221 at the J5 VDDA/VDD pins; C222/C223 at the J6 VDD pin."
- note removed: "SCS active-HIGH, LSB-first, <=2 MHz; write-only (no MISO)."

Commit message: add 7x SK6812 RGBW NeoPixel chain, drop panel LED string
- 5 status pixels (bell/alarm/clock/vol/batt) + 2 dial-wash pixels on the
  PCB, 5 V rail, one data GPIO (IO7 -> RMT) via SN74AHCT1G125 buffer
- panel string (Cree CLM3C x12) + its AO3400A + LEDC channel removed
- led.md rewritten for the new wake-COB + NeoPixel architecture

Co-Authored-By: Claude Fable 5 <noreply@anthropic.com>
Parts:
- removed J8: Panel LEDs 5V (CLM3C x12), Connector_JST:JST_PH_B2B-PH-K_1x02_P2.00mm_Vertical, symbol Connector_Generic:Conn_01x02
- removed Q5: AO3400A, Package_TO_SOT_SMD:SOT-23, symbol clock:AO3400A
- removed R102: 100R, Resistor_SMD:R_0603_1608Metric, symbol Device:R
- removed R103: 10k, Resistor_SMD:R_0603_1608Metric, symbol Device:R
- added C230, C231, C232, C233, C234, C235, C236, C238: 100nF, Capacitor_SMD:C_0603_1608Metric, symbol Device:C
- added C237: 100uF, Capacitor_SMD:CP_Elec_6.3x7.7, symbol Device:C_Polarized
- added D40, D41, D42, D43, D44, D45, D46: SK6812RGBW, LED_SMD:LED_SK6812_PLCC4_5.0x5.0mm_P3.2mm, symbol LED:SK6812
- added R110: 330R, Resistor_SMD:R_0603_1608Metric, symbol Device:R
- added U15: SN74AHCT1G125, Package_TO_SOT_SMD:SOT-23-5, symbol clock:74AHCT1G125
Connections:
- net +5V: now also C230.1, C231.1, C232.1, C233.1, C234.1, C235.1, C236.1, C237.1, C238.1, D40.3 (VDD), D41.3 (VDD), D42.3 (VDD), D43.3 (VDD), D44.3 (VDD), D45.3 (VDD), D46.3 (VDD), U15.5 (VCC)
- net GND: now also C230.2, C231.2, C232.2, C233.2, C234.2, C235.2, C236.2, C237.2, C238.2, D40.1 (VSS), D41.1 (VSS), D42.1 (VSS), D43.1 (VSS), D44.1 (VSS), D45.1 (VSS), D46.1 (VSS), U15.1, U15.3 (GND)
- net PANEL_PWM renamed NEOPIX_DATA
- net NEOPIX_DATA: now also U15.2
- new net: D40.2 (DIN), R110.2
- new net: D40.4 (DOUT), D41.2 (DIN)
- new net: D45.4 (DOUT), D46.2 (DIN)
- new net: D42.4 (DOUT), D43.2 (DIN)
- new net: D43.4 (DOUT), D44.2 (DIN)
- new net: D41.4 (DOUT), D42.2 (DIN)
- new net: D44.4 (DOUT), D45.2 (DIN)
- new net: R110.1, U15.4
- no-connect marks 18 -> 19
Other:
- note added: "(SK6812 VIH = 0.7*VDD = 3.5 V). <=0.6 A worst-case all-white."
- note added: "6-7 = dial wash. One RMT data line; AHCT buffer lifts 3V3 -> 5 V"
- note added: "ALARM"
- note added: "BATT"
- note added: "BELL"
- note added: "CLOCK"
- note added: "DIAL1"
- note added: "DIAL2"
- note added: "LED - wake COB drivers (12 V, plugged-only)"
- note added: "Layout: status row pitch = face-plate hole pitch; C230-236 one at each"
- note added: "Pixels 1-5 = status row behind the face holes (red/white semantics),"
- note added: "STATUS + DIAL NEOPIXELS - 7x SK6812 RGBW (5 V)"
- note added: "VOL"
- note added: "Wake COB strips are self-ballasted (12 V, plugged-only): firmware"
- note added: "gates their PWM off on battery. ~1 kHz, gamma; LED + audio <= ~12 W."
- note added: "pixel VDD; C237 bulk + R110 + U15 at the chain head."
- note removed: "LED DRIVERS — panel (5 V always) + wake COB (12 V plugged)"
- note removed: "Wake COB strips are self-ballasted (12 V). Panel string: one series R per LED,"
- note removed: "on the LED board. ~1 kHz PWM, gamma-corrected; wake channels plugged-only."

Commit message: knob: EM14 optical encoder + Kilo aluminum knob on host GPIO
- Bourns EM14A0D-C24-L064S (optical, no detent, 64 CPR, push, 5 V) under
  a Kilo OEJNI-90-1-5 machined knob (1/4in bore = EM14 shaft)
- J10 -> JST SH 1x06 (GND/+5V/A/B/SW/GND); A/B via 100k/200k dividers to
  IO47/48 (PCNT); ENC_SW -> IO17 host IRQ w/ 10k PU + 100nF debounce
- BTN1-3 + expander ENC_SW dropped (GPA3-6 freed; GPA3 reserved for the
  radio toggle); IO17 renamed from LCD_CS

Co-Authored-By: Claude Fable 5 <noreply@anthropic.com>
Parts:
- removed J10: UI: EC11 + 3 buttons (off-board), Connector_JST:JST_SH_SM08B-SRSS-TB_1x08-1MP_P1.00mm_Horizontal, symbol Connector_Generic:Conn_01x08
- removed R100, R101: 10k, Resistor_SMD:R_0603_1608Metric, symbol Device:R
- added C239: 100nF, Capacitor_SMD:C_0603_1608Metric, symbol Device:C
- added J10: Knob: EM14 enc+SW (top face), Connector_JST:JST_SH_SM06B-SRSS-TB_1x06-1MP_P1.00mm_Horizontal, symbol Connector_Generic:Conn_01x06
- added R111, R112: 100k, Resistor_SMD:R_0603_1608Metric, symbol Device:R
- added R113: 10k, Resistor_SMD:R_0603_1608Metric, symbol Device:R
- added R114, R115: 200k, Resistor_SMD:R_0603_1608Metric, symbol Device:R
Connections:
- net +3V3: now also R113.1
- net +5V: now also J10.2 (Pin_2)
- net GND: now also C239.2, J10.1 (Pin_1), J10.6 (Pin_6), R114.2, R115.2
- net at U8.25 (IO48_ENC_B): now also R112.1, R115.1
- net at U8.24 (IO47_ENC_A): now also R111.1, R114.1
- net ENC_SW: now reaches U8.10 (IO17_ENC_SW)
- net ENC_SW: now also C239.1, J10.5 (Pin_5), R113.2
- new net: J10.3 (Pin_3), R111.2
- new net: J10.4 (Pin_4), R112.2
- no-connect marks 19 -> 22
Other:
- note added: "(optical, 64 CPR, no detent, push) on the top face -> J10 SH cable. A/B are 5 V"
- note added: "INT: any GPA/GPB change -> IO44 (IOCON.MIRROR=1). Knob = EM14A0D-C24-L064S"
- note added: "IO EXPANDER (MCP23017 @0x20) + KNOB (EM14)"
- note added: "push-pull -> 100k/200k dividers -> PCNT IO47/48; SW -> 10k PU + 100n -> IO17 IRQ."
- note removed: "INT: any GPA/GPB change -> IO44 (IOCON.MIRROR=1). EC11 + buttons mount on the"
- note removed: "IO EXPANDER (MCP23017 @0x20) + ENCODER + BUTTONS"
- note removed: "Switch lines: MCP internal pull-ups + IOC. Encoder A/B -> PCNT (IO47/48), R100/R101 PU."
- note removed: "enclosure -> JST SH cable to J10 (1 GND, 2 ENC_A, 3 ENC_B, 4-6 BTN1-3, 7 ENC_SW, 8 GND)."

Commit message: radio-off toggle + vertical TH USB-C; sync docs to v0.19
- J11 (JST SH 1x02) -> MCP23017 GPA3 RADIO_OFF (rear Wi-Fi/BLE kill toggle)
- USB-C: USB4105 horizontal + Adafruit 6069 extension -> Same Sky
  UJ20-C-V-C-2-SMT-TR vertical (16-pin TH, port out the back wall; the
  suggested -C-1 is spec'd for 0.8 mm PCBs -> -C-2 for our 1.6 mm board;
  backorder at DigiKey 2026-07-19, GCT USB4145-03-0170-C = in-stock alt);
  custom TH footprint in clock.pretty (verify vs Same Sky DXF before fab)
- esp32.md / led.md / power.md / power_values.md / kicad/README.md /
  CLAUDE.md synced (pin map, expander map, rails, LED subsystem, BOM);
  datasheet/ intentionally untouched (display-era docs kept for reuse)

Co-Authored-By: Claude Fable 5 <noreply@anthropic.com>
Parts:
- added J11: Radio-off toggle (rear), Connector_JST:JST_SH_SM02B-SRSS-TB_1x02-1MP_P1.00mm_Horizontal, symbol Connector_Generic:Conn_01x02
- J1: value USB4105-GF-A -> UJ20-C-V-C-2-SMT-TR; footprint Connector_USB:USB_C_Receptacle_GCT_USB4105-xx-A_16P_TopMnt_Horizontal -> clock:SameSky_UJ20-C-V-C-2_USB_C_Vertical_TH
Connections:
- net GND: now also J11.2 (Pin_2)
- net at U13.24 (GPA3): now also J11.1 (Pin_1)
- no-connect marks 22 -> 21
Other:
- note added: "Off-board parts (SD card, sensors, speaker, wake-LED strips,"
- note added: "Vertical receptacle (TH pins) - port straight out the back wall."
- note added: "knob, radio toggle, cell) enter via connectors J1..J11 / BT1."
- note removed: "Off-board parts (display, SD, sensors, speaker, motor, LED"
- note removed: "strips, encoder+buttons, cell) enter via connectors J1..J10 / BT1."
