File: kicad/clock.kicad_sch (KiCad schematic)
At the start: 182 parts, among them J1 USB4160-03-0230-C, J10 Knob: EM14 enc+SW (top face), J11 Radio-off toggle (rear), J12 NeoPixel ext (5V/DATA/GND, po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, J2 PROG, J3 Speaker DMA58-4 (4R), J6 DM3AT-SF-PEJM5, J7 Sensor board (BME688+TSL2591+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, J9 Wake COB 12V (warm+cool), M1 X40.879, Q1 2N7002, Q2 AO3401A, Q3 2N7002, Q4 AO3401A, Q6 AO3400A, Q7 AO3400A, Q8 2N7002, Q9 AO3401A, SW1 RESET, SW2 BOOT, U1 CH224K, U10 LTC4412ES6, U11 TB6612FNG, U12 TB6612FNG, U13 MCP23017, U14 QRE1113GR, U15 SN74AHCT1G125, U16 USBLC6-2SC6, U2 LT3652EMSE, U3 HY2111-GB, U4 AOSD32334C, U5 TPS61023, U6 TLV62569DBVR, U7 TPS55340PWPR, U8 ESP32-S3-WROOM-1-N16R8, U9 TAS5760MDAPR, Y1 32.768kHz

Commit message: schematic ready rev0.1
Other:
- company: (none) -> Tibo Mauron
- title: Wooden Smart Clock — main board -> Wooden Clock - main board
Changed lines of the file:
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@@
 	(paper "A1")
 	(title_block
-		(title "Wooden Smart Clock — main board")
+		(title "Wooden Clock - main board")
 		(date "2026-07-14")
-		(rev "A")
+		(rev "0.1")
+		(company "Tibo Mauron")
 	)
 	(rectangle
@@
 	(rectangle
 		(start 610 110)
-		(end 835 180)
+		(end 826.77 180)
 		(stroke
 			(width 0.2)
@@
 	(rectangle
 		(start 610 405)
-		(end 835 585)
+		(end 826.77 581.66)
 		(stroke
 			(width 0.2)
@@
 	(rectangle
 		(start 405 415)
-		(end 595 585)
+		(end 595 579.12)
 		(stroke
 			(width 0.2)
@@
 	(rectangle
 		(start 610 190)
-		(end 835 385)
+		(end 826.77 385)
 		(stroke
 			(width 0.2)
@@
 	(text "STORAGE — microSD (DM3AT), SPI2 dedicated"
 		(exclude_from_sim no)
-		(at 612.5 114.2 0)
+		(at 685.292 113.538 0)
 		(effects
 			(font
@@
 	(text "INT: any GPA/GPB change -> IO44 (IOCON.MIRROR=1).  Knob = EM14A0D-C24-L064S"
 		(exclude_from_sim no)
-		(at 410 571 0)
+		(at 409.956 561.666 0)
 		(effects
 			(font
@@
 	(text "IO EXPANDER (MCP23017 @0x20) + KNOB (EM14)"
 		(exclude_from_sim no)
-		(at 407.5 419.2 0)
+		(at 484.632 419.608 0)
 		(effects
 			(font
@@
 	(text "CFG1=56k -> 15 V PDO; falls back to 5 V (charger idles <11.2 V)."
 		(exclude_from_sim no)
-		(at 20 141 0)
+		(at 19.558 138.35 0)
 		(effects
 			(font
@@
 	(text "IO35-37 reserved by the octal PSRAM (N16R8).  Straps: IO0 high; IO45/46 low via"
 		(exclude_from_sim no)
-		(at 410 48 0)
+		(at 408.178 49.022 0)
 		(effects
 			(font
@@
 	(text "D+/D- = native USB-JTAG (IO19/20). Vertical - port out the back wall."
 		(exclude_from_sim no)
-		(at 20 150.5 0)
+		(at 19.558 147.85 0)
 		(effects
 			(font
@@
 	(text "Li-ion 18650 ONLY - 2.5-4.2 V"
 		(exclude_from_sim no)
-		(at 25 190 0)
+		(at 21.844 188.722 0)
 		(effects
 			(font
@@
 	(text "AUDIO — TAS5760M PBTL + LC filter + PVDD mux (12V/5V)"
 		(exclude_from_sim no)
-		(at 612.5 194.2 0)
+		(at 651.764 195.072 0)
 		(effects
 			(font
@@
 	(text "PWM-on-IN microstepping: MCPWM waveforms on AIN/BIN, PWMA/B tied high."
 		(exclude_from_sim no)
-		(at 615 575 0)
+		(at 612.14 574.294 0)
 		(effects
 			(font
@@
 	(text "their wake gate nets + internal PD; IO3 internal.  Flash+console+JTAG = USB-CDC (IO19/20)."
 		(exclude_from_sim no)
-		(at 410 53 0)
+		(at 408.432 53.848 0)
 		(effects
 			(font
@@
 	(text "Layout: C222/C223 at the J6 VDD pin."
 		(exclude_from_sim no)
-		(at 688.34 130 0)
+		(at 785.876 139.446 0)
 		(effects
 			(font
@@
 	(text "1x02 (pre-crimped AxxZR cables).  A/B 5 V -> 100k/200k div -> PCNT; SW -> IO17 IRQ."
 		(exclude_from_sim no)
-		(at 410 580 0)
+		(at 409.956 570.666 0)
 		(effects
 			(font
@@
 	(text "MOTOR — 2x TB6612FNG -> X40.879 dual-shaft stepper"
 		(exclude_from_sim no)
-		(at 612.5 409.2 0)
+		(at 625.348 409.194 0)
 		(effects
 			(font
@@
 	(text "CH224K DP/DM shorted = PD-only; Type-C D± go to the MCU."
 		(exclude_from_sim no)
-		(at 20 136 0)
+		(at 19.558 133.35 0)
 		(effects
 			(font
@@
 	(text "Layout: each driver's 10uF+100nF go at its VM pins, the 100nF at its VCC pin."
 		(exclude_from_sim no)
-		(at 615 415 0)
+		(at 625.602 414.782 0)
 		(effects
 			(font
@@
 	(text "USB 2.0 subset of the 24-pin USB4160 (SS pads unconnected);"
 		(exclude_from_sim no)
-		(at 20 146 0)
+		(at 19.558 143.35 0)
 		(effects
 			(font
@@
 	(text "(optical, 64 CPR, no detent, push) on the top face.  J7/J10 = JST ZH 1x06, J11 = ZH"
 		(exclude_from_sim no)
-		(at 410 575.5 0)
+		(at 409.956 566.166 0)
 		(effects
 			(font
@@
 	(text "STEP_STBY (expander GPA1) low at boot -> drivers off. Coil map: esp32.md."
 		(exclude_from_sim no)
-		(at 615 579.5 0)
+		(at 612.394 577.596 0)
 		(effects
 			(font
@@
 	)
 	(junction
-		(at 73.66 228.6)
-		(diameter 0)
-		(color 0 0 0 0)
-	)
-	(junction
 		(at 474.98 106.68)
 		(diameter 0)
@@
 	)
 	(junction
-		(at 73.66 224.79)
-		(diameter 0)
-		(color 0 0 0 0)
-	)
-	(junction
 		(at 332.74 121.92)
 		(diameter 0)
@@
 	)
 	(junction
-		(at 237.49 332.74)
-		(diameter 0)
-		(color 0 0 0 0)
-	)
-	(junction
 		(at 91.44 247.65)
 		(diameter 0)
@@
 	)
 	(junction
+		(at 77.47 224.79)
+		(diameter 0)
+		(color 0 0 0 0)
+	)
+	(junction
 		(at 468.63 92.71)
 		(diameter 0)
@@
 	(wire
 		(pts
-			(xy 311.15 320.04) (xy 281.94 320.04)
-		)
-		(stroke
-			(width 0)
-			(type default)
-		)
-	)
-	(wire
-		(pts
 			(xy 549.91 111.76) (xy 678.18 111.76)
 		)
@@
 	(wire
 		(pts
-			(xy 300.99 320.04) (xy 281.94 320.04)
-		)
-		(stroke
-			(width 0)
-			(type default)
-		)
-	)
-	(wire
-		(pts
 			(xy 175.26 317.5) (xy 237.49 317.5)
 		)
@@
 	(wire
 		(pts
-			(xy 73.66 228.6) (xy 73.66 219.71)
+			(xy 77.47 219.71) (xy 77.47 224.79)
 		)
 		(stroke
@@
 	(wire
 		(pts
+			(xy 77.47 224.79) (xy 77.47 228.6)
+		)
+		(stroke
+			(width 0)
+			(type default)
+		)
+	)
+	(wire
+		(pts
 			(xy 654.05 154.94) (xy 654.05 167.64)
 		)
@@
 	(wire
 		(pts
-			(xy 237.49 332.74) (xy 237.49 332.74)
-		)
-		(stroke
-			(width 0)
-			(type default)
-		)
-	)
-	(wire
-		(pts
 			(xy 695.96 568.96) (xy 695.96 571.5)
 		)
@@
 	(wire
 		(pts
-			(xy 73.66 219.71) (xy 78.74 219.71)
-		)
-		(stroke
-			(width 0)
-			(type default)
-		)
-	)
-	(wire
-		(pts
 			(xy 695.96 441.96) (xy 695.96 439.42)
 		)
@@
 	(wire
 		(pts
-			(xy 73.66 224.79) (xy 73.66 228.6)
-		)
-		(stroke
-			(width 0)
-			(type default)
-		)
-	)
-	(wire
-		(pts
 			(xy 695.96 492.76) (xy 695.96 495.3)
 		)
@@
 	(wire
 		(pts
-			(xy 67.31 224.79) (xy 73.66 224.79)
+			(xy 67.31 224.79) (xy 77.47 224.79)
 		)
 		(stroke
@@
 	(wire
 		(pts
-			(xy 290.83 320.04) (xy 281.94 320.04)
+			(xy 281.94 320.04) (xy 311.15 320.04)
 		)
 		(stroke
@@
 	(wire
 		(pts
-			(xy 83.82 228.6) (xy 73.66 228.6)
+			(xy 83.82 228.6) (xy 77.47 228.6)
 		)
 		(stroke
@@
 	(global_label "VBAT_DIV_EN"
 		(shape bidirectional)
-		(at 78.74 219.71 180)
+		(at 77.47 219.71 180)
 		(effects
 			(font
@@
 		)
 		(property "Intersheetrefs" "${INTERSHEET_REFS}"
-			(at 78.74 219.71 0)
+			(at 77.47 219.71 0)
 			(hide yes)
 			(show_name no)

Commit message: fix BOM list
Parts:
- BT1: MPN (none) -> 1043; Manufacturer (none) -> Keystone Electronics; Package (none) -> TH holder, 18650
- C1, C108, C144, C160, C165, C167, C171: MPN (none) -> CL10B105KA8NNNC; Manufacturer (none) -> Samsung Electro-Mechanics; Notes (none) -> Substitution OK - same value/tolerance/voltage/dielectric/s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; Package (none) -> 0603
- C100, C101, C106, C120, C124, C127, C140, C162, C200, C210, C222: MPN (none) -> CL21A106KAYNNNE; Manufacturer (none) -> Samsung Electro-Mechanics; Notes (none) -> Substitution OK - same value/tolerance/voltage/dielectric/s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; Package (none) -> 0805
- C102, C104, C109, C110, C128, C134, C142, C143, C161, C163, C164, C166, C170, C186, C201, C202, C211, C212, C223, C230, C231, C238, C239, C240, C241: MPN (none) -> CL10B104KB8NNNC; Manufacturer (none) -> Samsung Electro-Mechanics; Notes (none) -> Substitution OK - same value/tolerance/voltage/dielectric/s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; Package (none) -> 0603
- C105: MPN (none) -> CL10C220JB8NNNC; Manufacturer (none) -> Samsung Electro-Mechanics; Notes (none) -> Substitution OK - same value/tolerance/voltage/dielectric/s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; Package (none) -> 0603
- C107, C129, C237: MPN (none) -> EEE-FK1C101P; Manufacturer (none) -> Panasonic; Notes (none) -> Substitution OK - same value/tolerance/voltage/dielectric/s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; Package (none) -> SMD radial can D6.3xL6.1mm
- C121, C122, C125, C141: MPN (none) -> CL21A226MOQNNNE; Manufacturer (none) -> Samsung Electro-Mechanics; Notes (none) -> Substitution OK - same value/tolerance/voltage/dielectric/s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; Package (none) -> 0805
- C123: MPN (none) -> CL10C221JB8NNNC; Manufacturer (none) -> Samsung Electro-Mechanics; Notes (none) -> Substitution OK - same value/tolerance/voltage/dielectric/s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; Package (none) -> 0603
- C126: MPN (none) -> CL10C6R8BB8NNNC; Manufacturer (none) -> Samsung Electro-Mechanics; Notes (none) -> Substitution OK - same value/tolerance/voltage/dielectric/s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; Package (none) -> 0603
- C130, C131, C132: MPN (none) -> GRM32ER71E226KE15L; Manufacturer (none) -> Murata Electronics; Notes (none) -> Substitution OK - same value/tolerance/voltage/dielectric/s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; Package (none) -> 1210
- C133: MPN (none) -> CL10B473KB8NNNC; Manufacturer (none) -> Samsung Electro-Mechanics; Notes (none) -> Substitution OK - same value/tolerance/voltage/dielectric/s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; Package (none) -> 0603
- C135: MPN (none) -> CL10C101JB8NNNC; Manufacturer (none) -> Samsung Electro-Mechanics; Notes (none) -> Substitution OK - same value/tolerance/voltage/dielectric/s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; Package (none) -> 0603
- C145, C146: MPN (none) -> CL10C180JB8NNNC; Manufacturer (none) -> Samsung Electro-Mechanics; Notes (none) -> Substitution OK - same value/tolerance/voltage/dielectric/s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; Package (none) -> 0603
- C172: value 220uF -> 100uF; MPN (none) -> 25TZV100M6.3X8; Manufacturer (none) -> Rubycon; Notes (none) -> PVDD bulk. Was 220uF: no tier-1 220uF >=16V exists in a D6.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; Package (none) -> SMD radial can D6.3xL8.0mm
- C180, C181, C182, C183: MPN (none) -> CL10B224KA8NNNC; Manufacturer (none) -> Samsung Electro-Mechanics; Notes (none) -> Substitution OK - same value/tolerance/voltage/dielectric/s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; Package (none) -> 0603
- C184, C185: MPN (none) -> C0805C684K5RACTU; Manufacturer (none) -> KEMET; Notes (none) -> Substitution OK - same value/tolerance/voltage/dielectric/s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; Package (none) -> 0805
- D1: MPN (none) -> SMAJ22CA; Manufacturer (none) -> Littelfuse; Package (none) -> DO-214AC (SMA)
- D10: MPN (none) -> BAT46W-E3-08; Manufacturer (none) -> Vishay; Package (none) -> SOD-123
- D11, D20, D30: MPN (none) -> B340A-13-F; Manufacturer (none) -> Diodes Incorporated; Package (none) -> DO-214AC (SMA)
- D12: MPN (none) -> SMAJ5.0CA; Manufacturer (none) -> Littelfuse; Package (none) -> DO-214AC (SMA)
- D13: MPN (none) -> BAT42W-E3-08; Manufacturer (none) -> Vishay; Package (none) -> SOD-123
- D40, D41: MPN (none) -> SK6812RGBW; Manufacturer (none) -> Opsco Optoelectronics; Notes (none) -> = Adafruit 2758 10-pack (DigiKey 6134706); any SK6812 RGBW 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; Package (none) -> PLCC-4 5.0x5.0mm
- F1: MPN (none) -> SDF-DF077S; Manufacturer (none) -> Cantherm; Notes (none) -> Solder >=3 mm from the body and heatsink the lead; Package (none) -> Radial D4.0mm, axial AWG18 leads
- J1: MPN (none) -> USB4160-03-0230-C; Manufacturer (none) -> GCT; Notes (none) -> USB 2.0 subset wired (VBUS/GND/CC/D+/D-); SS pads unconnect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; Package (none) -> SMT vertical, 24-pin + 4 stakes
- J10, J7: MPN (none) -> B6B-ZR(LF)(SN); Manufacturer (none) -> JST Sales America; Package (none) -> JST ZH 1.50mm 6-pos TH vertical
- J11: MPN (none) -> B2B-ZR(LF)(SN); Manufacturer (none) -> JST Sales America; Package (none) -> JST ZH 1.50mm 2-pos TH vertical
- J12, J9: MPN (none) -> B3B-PH-K-S(LF)(SN); Manufacturer (none) -> JST Sales America; Package (none) -> JST PH 2.00mm 3-pos TH vertical
- J2: MPN (none) -> PRPC004SAAN-RC; Manufacturer (none) -> Sullins Connector Solutions; Package (none) -> 1x04 2.54mm TH header
- J3: MPN (none) -> B2B-PH-K-S(LF)(SN); Manufacturer (none) -> JST Sales America; Package (none) -> JST PH 2.00mm 2-pos TH vertical
- J6: MPN (none) -> DM3AT-SF-PEJM5; Manufacturer (none) -> Hirose Electric; Package (none) -> SMT push-push, 8-pos
- L1, L5, L6: MPN (none) -> XAL4040-103MEC; Manufacturer (none) -> Coilcraft; Package (none) -> SMD 4.0x4.0x4.0mm
- L2: MPN (none) -> XAL4020-102MEC; Manufacturer (none) -> Coilcraft; Package (none) -> SMD 4.0x4.0x2.1mm
- L3: MPN (none) -> XAL4020-222MEC; Manufacturer (none) -> Coilcraft; Package (none) -> SMD 4.0x4.0x2.1mm
- L4: MPN (none) -> XGL5050-472MEC; Manufacturer (none) -> Coilcraft; Notes (none) -> On the XAL5050 land - verified 2026-07-27: identical to the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; Package (none) -> SMD 5.3x5.5x5.0mm
- M1: MPN (none) -> X40.879; Manufacturer (none) -> Juken Swiss Technology; Notes (none) -> Custom footprint; shafts pass through the board. Long lead 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; Package (none) -> TH, 8 pins, dual coaxial shaft
- Q1, Q3, Q8: MPN (none) -> 2N7002LT1G; Manufacturer (none) -> onsemi; Package (none) -> SOT-23
- Q2, Q4, Q9: MPN (none) -> AO3401A; Manufacturer (none) -> Alpha & Omega Semiconductor; Package (none) -> SOT-23
- Q6, Q7: MPN (none) -> AO3400A; Manufacturer (none) -> Alpha & Omega Semiconductor; Package (none) -> SOT-23
- R1: MPN (none) -> RC0603FR-071KL; Manufacturer (none) -> YAGEO; Notes (none) -> Substitution OK - same value/tolerance/voltage/dielectric/s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; Package (none) -> 0603
- R10: MPN (none) -> RC0603FR-07316KL; Manufacturer (none) -> YAGEO; Notes (none) -> Substitution OK - same value/tolerance/voltage/dielectric/s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; Package (none) -> 0603
- R104, R106, R20: MPN (none) -> RC0603FR-07100RL; Manufacturer (none) -> YAGEO; Notes (none) -> Substitution OK - same value/tolerance/voltage/dielectric/s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; Package (none) -> 0603
- R105, R107, R113, R12, R13, R2, R4, R46, R50, R51, R60, R62, R70, R71, R72, R93, R94, R97, R99: MPN (none) -> RC0603FR-0710KL; Manufacturer (none) -> YAGEO; Notes (none) -> Substitution OK - same value/tolerance/voltage/dielectric/s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; Package (none) -> 0603
- R11, R111, R112, R19, R22, R23, R24, R25, R26, R27, R41, R43, R44, R63: MPN (none) -> RC0603FR-07100KL; Manufacturer (none) -> YAGEO; Notes (none) -> Substitution OK - same value/tolerance/voltage/dielectric/s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; Package (none) -> 0603
- R110: MPN (none) -> RC0603FR-07330RL; Manufacturer (none) -> YAGEO; Notes (none) -> Substitution OK - same value/tolerance/voltage/dielectric/s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; Package (none) -> 0603
- R114, R115, R15: MPN (none) -> RC0603FR-07200KL; Manufacturer (none) -> YAGEO; Notes (none) -> Substitution OK - same value/tolerance/voltage/dielectric/s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; Package (none) -> 0603
- R14: MPN (none) -> RC0603FR-0745K3L; Manufacturer (none) -> YAGEO; Notes (none) -> Substitution OK - same value/tolerance/voltage/dielectric/s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; Package (none) -> 0603
- R16: MPN (none) -> RC0603FR-07976KL; Manufacturer (none) -> YAGEO; Notes (none) -> Substitution OK - same value/tolerance/voltage/dielectric/s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; Package (none) -> 0603
- R17: MPN (none) -> RC0603FR-07909RL; Manufacturer (none) -> YAGEO; Notes (none) -> Substitution OK - same value/tolerance/voltage/dielectric/s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; Package (none) -> 0603
- R18: MPN (none) -> WSL2010R1000FEA18; Manufacturer (none) -> Vishay Dale; Notes (none) -> LT3652 sense; dissipates 0.1 W at I_CHG 1 A. The ...FEA18 s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; Package (none) -> 2010
- R21: MPN (none) -> RC0603FR-072KL; Manufacturer (none) -> YAGEO; Notes (none) -> Substitution OK - same value/tolerance/voltage/dielectric/s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; Package (none) -> 0603
- R3: MPN (none) -> RC0603FR-0756KL; Manufacturer (none) -> YAGEO; Notes (none) -> Substitution OK - same value/tolerance/voltage/dielectric/s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; Package (none) -> 0603
- R40: MPN (none) -> RC0603FR-07732KL; Manufacturer (none) -> YAGEO; Notes (none) -> Substitution OK - same value/tolerance/voltage/dielectric/s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; Package (none) -> 0603
- R42: MPN (none) -> RC0603FR-07453KL; Manufacturer (none) -> YAGEO; Notes (none) -> Substitution OK - same value/tolerance/voltage/dielectric/s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; Package (none) -> 0603
- R45: MPN (none) -> RC0603FR-0786K6L; Manufacturer (none) -> YAGEO; Notes (none) -> Substitution OK - same value/tolerance/voltage/dielectric/s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; Package (none) -> 0603
- R47: MPN (none) -> RC0603FR-0795K3L; Manufacturer (none) -> YAGEO; Notes (none) -> Substitution OK - same value/tolerance/voltage/dielectric/s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; Package (none) -> 0603
- R48: MPN (none) -> RC0603FR-072K55L; Manufacturer (none) -> YAGEO; Notes (none) -> Substitution OK - same value/tolerance/voltage/dielectric/s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; Package (none) -> 0603
- R61, R90, R91, R92: MPN (none) -> RC0603JR-070RL; Manufacturer (none) -> YAGEO; Notes (none) -> Substitution OK - same value/tolerance/voltage/dielectric/s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; Package (none) -> 0603
- R95, R96: MPN (none) -> RC0603FR-074K7L; Manufacturer (none) -> YAGEO; Notes (none) -> Substitution OK - same value/tolerance/voltage/dielectric/s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; Package (none) -> 0603
- R98: MPN (none) -> RC0603FR-07150RL; Manufacturer (none) -> YAGEO; Notes (none) -> Substitution OK - same value/tolerance/voltage/dielectric/s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; Package (none) -> 0603
- RT1: value 10k -> 10k NTC; MPN (none) -> NCP18XH103F03RB; Manufacturer (none) -> Murata Electronics; Notes (none) -> NTC, not a resistor - do not merge with the 10k line; Package (none) -> 0603
- SW1, SW2: MPN (none) -> RS-282G05A3-SM RT; Manufacturer (none) -> C&K; Package (none) -> SMD tactile 4.2x3.2mm
- U1: MPN (none) -> CH224K; Manufacturer (none) -> WCH (Nanjing Qinheng); Notes (none) -> Not stocked at DigiKey - LCSC C970725; Package (none) -> ESSOP-10 (SSOP-10, EP)
- U10: MPN (none) -> LTC4412ES6#TRPBF; Manufacturer (none) -> Analog Devices; Package (none) -> TSOT-23-6
- U11, U12: MPN (none) -> TB6612FNG,C,8,EL; Manufacturer (none) -> Toshiba; Package (none) -> 24-SSOP
- U13: MPN (none) -> MCP23017-E/SS; Manufacturer (none) -> Microchip Technology; Notes (none) -> SSOP-28 land (README §16b quotes the -E/SO SOIC-28W order c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; Package (none) -> 28-SSOP
- U14: MPN (none) -> QRE1113GR; Manufacturer (none) -> onsemi; Package (none) -> SMD gull-wing 4-lead
- U15: MPN (none) -> SN74AHCT1G125DBVR; Manufacturer (none) -> Texas Instruments; Package (none) -> SOT-23-5
- U16: MPN (none) -> USBLC6-2SC6; Manufacturer (none) -> STMicroelectronics; Package (none) -> SOT-23-6
- U2: MPN (none) -> LT3652EMSE#PBF; Manufacturer (none) -> Analog Devices; Package (none) -> 12-MSOP-EP
- U3: MPN (none) -> HY2111-GB; Manufacturer (none) -> HYCON Technology; Notes (none) -> Not stocked at DigiKey - LCSC C82747; Package (none) -> SOT-23-6
- U4: MPN (none) -> AOSD32334C; Manufacturer (none) -> Alpha & Omega Semiconductor; Package (none) -> 8-SOIC
- U5: MPN (none) -> TPS61023DRLR; Manufacturer (none) -> Texas Instruments; Package (none) -> SOT-563
- U6: MPN (none) -> TLV62569DBVR; Manufacturer (none) -> Texas Instruments; Notes (none) -> DBV = SOT-23-5 (README §16b says SOT-23-6 - README is wrong); Package (none) -> SOT-23-5
- U7: MPN (none) -> TPS55340PWPR; Manufacturer (none) -> Texas Instruments; Package (none) -> 14-HTSSOP-EP (PWP)
- U8: MPN (none) -> ESP32-S3-WROOM-1-N16R8; Manufacturer (none) -> Espressif Systems; Package (none) -> SMD module 18x25.5mm, castellated
- U9: MPN (none) -> TAS5760MDAPR; Manufacturer (none) -> Texas Instruments; Package (none) -> 32-HTSSOP-EP (DAP)
- Y1: MPN (none) -> ABS07-32.768KHZ-T; Manufacturer (none) -> Abracon; Package (none) -> SMD 3.2x1.5mm 2-pin
