File: kicad/clock.kicad_sch (KiCad schematic)
At the start: 183 parts, among them J1 USB4160-03-0230-C, J10 Knob: EM14 enc+SW (top face), J11 Radio-off toggle (rear), J12 NeoPixel ext (5V/DATA/GND, po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, J2 PROG, J3 Speaker DMA58-4 (4R), J6 DM3AT-SF-PEJM5, J7 Sensor board (BME688+TSL2591+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, J9 Wake COB 12V (warm+cool), M1 X40.879, Q1 2N7002, Q2 AO3401A, Q3 2N7002, Q4 AO3401A, Q6 AO3400A, Q7 AO3400A, Q8 2N7002, Q9 AO3401A, SW1 RESET, SW2 BOOT, U1 CH224K, U10 LTC4412ES6, U11 TB6612FNG, U12 TB6612FNG, U13 MCP23017, U14 QRE1113GR, U15 SN74AHCT1G125, U16 USBLC6-2SC6, U2 LT3652EMSE, U3 HY2111-GB, U4 AOSD32334C, U5 TPS61023, U6 TLV62569DBVR, U7 TPS55340PWPR, U8 ESP32-S3-WROOM-1-N16R8, U9 TAS5760MDAPR, Y1 32.768kHz

Commit message: manual modifications
Other:
- company: (none) -> Tibo
- title: Wooden Smart Clock — main board -> Wooden Clock - main board
- moved on the sheet: D14
