File: kicad2/clock.kicad_sch (KiCad schematic)
At the start: 88 parts, among them J1 USB4105-GF-A, J8 Panel LEDs 5V (CLM3C x12), J9 Wake COB 12V (warm+cool), Q1 2N7002, Q2 AO3401A, Q3 2N7002, Q5 AO3400A, Q6 AO3400A, Q7 AO3400A, U1 CH224K, U2 LT3652EMSE, U3 AP9101CK6-BX, U4 AOSD32334C, U5 TPS61023, U6 TLV62569DBVR, U7 TPS55340PWPR

Commit message: kicad2, pass 2
Parts:
- added C140, C162, C200, C210, C222: 10uF, Capacitor_SMD:C_0805_2012Metric, symbol Device:C
- added C141: 22uF, Capacitor_SMD:C_0805_2012Metric, symbol Device:C
- added C142, C143, C161, C164, C166, C170, C186, C201, C202, C211, C212, C223, C240, C241: 100nF, Capacitor_SMD:C_0603_1608Metric, symbol Device:C
- added C144, C160, C165, C167, C171, C220, C221: 1uF, Capacitor_SMD:C_0603_1608Metric, symbol Device:C
- added C145, C146: 18pF, Capacitor_SMD:C_0603_1608Metric, symbol Device:C
- added C172: 220uF, Capacitor_SMD:CP_Elec_6.3x7.7, symbol Device:C_Polarized
- added C180, C181, C182, C183: 33nF, Capacitor_SMD:C_0603_1608Metric, symbol Device:C
- added C184, C185: 0.68uF, Capacitor_SMD:C_0805_2012Metric, symbol Device:C
- added D30: SS34, Diode_SMD:D_SMA, symbol Device:D_Schottky
- added J2: PROG, Connector_PinHeader_2.54mm:PinHeader_1x04_P2.54mm_Vertical, symbol Connector_Generic:Conn_01x04
- added J3: Speaker DMA58-4 (4R), Connector_JST:JST_PH_B2B-PH-K_1x02_P2.00mm_Vertical, symbol Connector_Generic:Conn_01x02
- added J4: X40.879 stepper (1e-4e, 1i-4i), Connector_JST:JST_PH_B8B-PH-K_1x08_P2.00mm_Vertical, symbol Connector_Generic:Conn_01x08
- added J5: LS032B7DD02 (FH34SRJ-10S), Connector_FFC-FPC:Hirose_FH34SRJ-10S-0.5SH_1x10-1MP_P0.50mm_Horizontal, symbol Connector_Generic:Conn_01x10
- added J6: DM3AT-SF-PEJM5, Connector_Card:microSD_HC_Hirose_DM3AT-SF-PEJM5, symbol clock:Micro_SD_Card_Det_Hirose_DM3AT
- added J7: Sensor board (BME688+TSL2591+LIS3DH), Connector_JST:JST_SH_SM05B-SRSS-TB_1x05-1MP_P1.00mm_Horizontal, symbol Connector_Generic:Conn_01x05
- added L5, L6: 10uH, Inductor_SMD:L_Coilcraft_XAL4030-XXX, symbol Device:L
- added Q4: AO3401A, Package_TO_SOT_SMD:SOT-23, symbol clock:AO3401A
- added R100, R101, R50, R51, R52, R60, R62, R70, R71, R72, R93, R94, R97, R99: 10k, Resistor_SMD:R_0603_1608Metric, symbol Device:R
- added R61, R90, R91, R92: 0R, Resistor_SMD:R_0603_1608Metric, symbol Device:R
- added R95, R96: 4.7k, Resistor_SMD:R_0603_1608Metric, symbol Device:R
- added R98: 150R, Resistor_SMD:R_0603_1608Metric, symbol Device:R
- added SW1: RESET, Button_Switch_SMD:SW_SPST_CK_RS282G05A3, symbol Switch:SW_Push
- added SW2: BOOT, Button_Switch_SMD:SW_SPST_CK_RS282G05A3, symbol Switch:SW_Push
- added SW3: EC11 encoder, Rotary_Encoder:RotaryEncoder_Alps_EC11E-Switch_Vertical_H20mm, symbol Device:RotaryEncoder_Switch
- added SW4: BTN1, Button_Switch_SMD:SW_SPST_CK_RS282G05A3, symbol Switch:SW_Push
- added SW5: BTN2, Button_Switch_SMD:SW_SPST_CK_RS282G05A3, symbol Switch:SW_Push
- added SW6: BTN3, Button_Switch_SMD:SW_SPST_CK_RS282G05A3, symbol Switch:SW_Push
- added U10: LTC4412ES6, Package_TO_SOT_SMD:SOT-23-6, symbol Power_Management:LTC4412xS6
- added U11, U12: TB6612FNG, Package_SO:SSOP-24_5.3x8.2mm_P0.65mm, symbol Driver_Motor:TB6612FNG
- added U13: MCP23017, Package_SO:SSOP-28_5.3x10.2mm_P0.65mm, symbol clock:MCP23017x-x-SS
- added U14: QRE1113, symbol Sensor_Proximity:QRE1113
- added U8: ESP32-S3-WROOM-1-N16R8, RF_Module:ESP32-S3-WROOM-1, symbol clock:ESP32S3_CLOCK
- added U9: TAS5760MDAPR, Package_SO:HTSSOP-32-1EP_6.1x11mm_P0.65mm_EP5.2x11mm_Mask4.11x4.36mm, symbol clock:TAS5760M
- added Y1: 32.768kHz, Crystal:Crystal_SMD_3215-2Pin_3.2x1.5mm, symbol Device:Crystal
Connections:
- net +12V: now also D30.2 (A)
- net +3V3: now also C140.1, C141.1, C142.1, C143.1, C161.1, C162.1, C202.1, C212.1, C222.1, C223.1, C240.1, J2.1 (Pin_1), J6.4 (VDD), J7.2 (Pin_2), R100.1, R101.1, R50.1, R51.1, R60.1, R62.2, R70.1, R71.1, R72.1, R93.1, R94.1, R95.1, R96.1, R97.1, R98.1, R99.1, U11.15 (PWMB), U11.20 (VCC), U11.23 (PWMA), U12.15 (PWMB), U12.20 (VCC), U12.23 (PWMA), U13.9 (V_{DD}), U8.2 (3V3), U9.1 (AVDD), U9.10 (DVDD)
- net +5V: now also C186.1, C200.1, C201.1, C210.1, C211.1, C220.1, C221.1, J5.6 (Pin_6), J5.7 (Pin_7), Q4.2 (S), U10.1 (VIN), U11.13 (VM2), U11.14 (VM3), U11.24 (VM1), U12.13 (VM2), U12.14 (VM3), U12.24 (VM1)
- net BOOST12_EN: now also U13.23 (GPA2)
- net CHRG: now also U13.2 (GPB1)
- net FAULT: now also U13.3 (GPB2)
- net FULLCHG_EN: now also U13.5 (GPB4)
- net GND: now also C140.2, C141.2, C142.2, C143.2, C144.2, C145.1, C146.1, C160.2, C161.2, C162.2, C164.2, C165.2, C166.2, C167.2, C170.2, C171.2, C172.2, C184.2, C185.2, C186.2, C200.2, C201.2, C202.2, C210.2, C211.2, C212.2, C220.2, C221.2, C222.2, C223.2, C240.2, C241.2, J2.2 (Pin_2), J5.10 (Pin_10), J5.4 (Pin_4), J5.8 (Pin_8), J5.9 (Pin_9), J6.6 (VSS), J6.SH (SHIELD), J7.1 (Pin_1), R52.2, R61.2, R90.2, R91.2, R92.2, SW1.1, SW2.1, SW3.C, SW3.S2, SW4.2, SW5.2, SW6.2, U10.2 (GND), U10.3 (CTL), U11.10 (PGND2), U11.18 (GND), U11.3 (PGND1), U11.4 (PGND1), U11.9 (PGND2), U12.10 (PGND2), U12.18 (GND), U12.3 (PGND1), U12.4 (PGND1), U12.9 (PGND2), U13.10 (V_{SS}), U14.2 (K), U14.4, U8.1 (GND), U8.40 (GND), U8.41 (GND), U9.18 (DGND), U9.22 (PGND), U9.27 (PGND), U9.31 (GGND), U9.33 (PAD)
- net PANEL_PWM: now also U8.7 (IO7 PWM_PANEL)
- net PD_PG: now also U13.1 (GPB0)
- net USB_DM: now also U8.13 (IO19 USB_D-)
- net USB_DP: now also U8.14 (IO20 USB_D+)
- net VBAT_DIV_EN: now also U13.6 (GPB5)
- net VBAT_SENSE: now also U8.39 (IO1 ADC_VBAT)
- net WAKE_COOL_PWM: now also R52.1, U8.16 (IO46 PWM_COOL)
- net WAKE_WARM_PWM: now also U8.26 (IO45 PWM_WARM)
- new net: R100.2, SW3.A, U8.24 (IO47 ENC_A)
- new net: R101.2, SW3.B, U8.25 (IO48 ENC_B)
- new net: SW3.S1, U13.27 (GPA6)
- new net: C181.1, C181.2, C183.1, C183.2, L6.1, U9.24 (BSTRPB-), U9.25 (BSTRPA-)
- new net: J4.1 (Pin_1), U11.5 (AO2), U11.6 (AO2)
- new net: J4.2 (Pin_2), U11.7 (BO2), U11.8 (BO2)
- new net: J4.3 (Pin_3), U11.11 (BO1), U11.12 (BO1)
- new net: J4.4 (Pin_4), U12.1 (AO1), U12.2 (AO1)
- new net: J4.5 (Pin_5), U12.5 (AO2), U12.6 (AO2)
- new net: J4.6 (Pin_6), U12.7 (BO2), U12.8 (BO2)
- new net: J4.7 (Pin_7), U12.11 (BO1), U12.12 (BO1)
- new net: C185.1, J3.2 (Pin_2), L6.2
- new net: Q4.1 (G), U10.5 (GATE)
- new net: R98.2, U14.1 (A)
- new net: C180.1, U9.30 (BSTRPA+)
- new net: C180.2, C182.1, C182.2, L5.1, U9.19 (BSTRPB+)
- new net: C164.1, C165.1, U9.3 (ANA_REG)
- new net: C167.1, U9.4 (VCOM)
- new net: C166.1, U9.5 (ANA_REF)
- new net: SW5.1, U13.25 (GPA4)
- new net: C146.2, U8.9 (IO16 XTAL_N), Y1.1
- new net: C145.2, U8.8 (IO15 XTAL_P), Y1.2
- new net: J2.4 (Pin_4), R51.2, SW2.2, U8.27 (IO0 BOOT)
- new net: SW4.1, U13.24 (GPA3)
- new net: C144.1, J2.3 (Pin_3), R50.2, SW1.2, U8.3 (EN)
- new net: J6.2 (DAT3/CD), R70.2, U8.11 (IO18 SD_CS)
- new net: C184.1, J3.1 (Pin_1), L5.2
- new net: J6.1 (DAT2), R71.2
- new net: J5.2 (Pin_2), J6.3 (CMD), U8.22 (IO14 MOSI)
- new net: J5.1 (Pin_1), J6.5 (CLK), U8.21 (IO13 SCLK)
- new net: J6.7 (DAT0), U8.23 (IO21 MISO)
- new net: J6.8 (DAT1), R72.2
- new net: R61.1, U9.13 (SPK_SLEEP/ADR)
- new net: R90.1, U13.15 (A0)
- new net: R60.2, U9.11 (SPK_GAIN0), U9.12 (SPK_GAIN1)
- new net: U8.37 (IO43 MCLK), U9.14 (MCLK)
- new net: U8.18 (IO10 BCLK), U9.15 (SCLK)
- new net: U8.20 (IO12 DOUT), U9.16 (SDIN)
- new net: U8.19 (IO11 LRCLK), U9.17 (LRCK)
- new net: C160.1, U9.2 (SFT_CLIP), U9.32 (GVDD_REG)
- new net: SW6.1, U13.26 (GPA5)
- new net: R92.1, U13.17 (A2)
- new net: U12.16 (BIN2), U8.34 (IO41 H_BIN2)
- new net: U12.17 (BIN1), U8.33 (IO40 H_BIN1)
- new net: U12.21 (AIN1), U8.31 (IO38 H_AIN1)
- new net: U12.22 (AIN2), U8.32 (IO39 H_AIN2)
- new net: R94.2, U13.19 (INTB), U13.20 (INTA), U8.36 (IO44 EXP_INT)
- new net: R91.1, U13.16 (A1)
- new net: J5.3 (Pin_3), U8.10 (IO17 LCD_CS)
- new net: R93.2, U13.18 (~{RESET})
- new net: U11.16 (BIN2), U8.15 (IO3 M_BIN2)
- new net: U11.21 (AIN1), U8.4 (IO4 M_AIN1)
- new net: U11.22 (AIN2), U8.5 (IO5 M_AIN2)
- new net: U11.17 (BIN1), U8.6 (IO6 M_BIN1)
- new net: U11.1 (AO1), U11.2 (AO1)
- new net HOME_OPTO: C241.1, R99.2, U14.3, U8.38 (IO2 ADC_HOME)
- new net I2C_SCL: J7.4 (Pin_4), R96.2, U13.12 (SCK), U8.17 (IO9 SCL), U9.9 (PBTL/SCL)
- new net I2C_SDA: J7.3 (Pin_3), R95.2, U13.13 (SDA), U8.12 (IO8 SDA), U9.8 (FREQ/SDA)
- new net LCD_DISP: J5.5 (Pin_5), U13.4 (GPB3)
- new net PVDD: C170.1, C171.1, C172.1, D30.1 (K), Q4.3 (D), U10.6 (SENSE)
- new net SENSOR_INT: J7.5 (Pin_5), R97.2, U8.35 (IO42 SENS_INT)
- new net SPK_FAULT: R62.1, U13.7 (GPB6), U9.6 (SPK_FAULT)
- new net SPK_SD: U13.21 (GPA0), U9.7 (SPK_SD)
- new net STEP_STBY: U11.19 (STBY), U12.19 (STBY), U13.22 (GPA1)
- no-connect marks 6 -> 16
Other:
- note added: "AUDIO — TAS5760M PBTL + LC filter + PVDD mux (12V/5V)"
- note added: "DISPLAY (LS032B7DD02, FPC) + microSD — shared SPI2"
- note added: "EXTMODE=L -> software VCOM (frame-inversion bit, >=1 Hz)."
- note added: "INT: any GPA/GPB change -> IO44 (IOCON.MIRROR=1). Buttons/encoder-switch"
- note added: "IO EXPANDER (MCP23017 @0x20) + ENCODER + BUTTONS"
- note added: "IO35-37 reserved by the octal PSRAM (N16R8). Straps: IO0 high, IO46 low (R52,"
- note added: "MCU — ESP32-S3-WROOM-1-N16R8 (Wi-Fi + BLE, native USB-JTAG)"
- note added: "MOTOR — 2x TB6612FNG -> X40.879 dual-shaft stepper"
- note added: "PBTL mono (reg 0x06[7]=1): OUTA||OUTB. MCLK 256fs ~12.288 MHz."
- note added: "PVDD auto-mux: 12 V wins when plugged; on battery Q4 ideal-diodes"
- note added: "PWM-on-IN microstepping: MCPWM waveforms on AIN/BIN, PWMA/B tied high."
- note added: "QRE1113 faces reflective tabs on the hand hubs (no magnets)."
- note added: "SCS active-HIGH, LSB-first, <=2 MHz; write-only (no MISO)."
- note added: "SENSORS (I2C off-board) + HAND-HOMING (QRE1113)"
- note added: "SPI mode: MSB-first, CS active-low, ~25 MHz. No card-detect (no spare GPIO)."
- note added: "STEP_STBY (expander GPA1) low at boot -> drivers off. Coil map: esp32.md."
- note added: "Sensor breakouts carry their own I2C pull-ups."
- note added: "at the LED block), IO3/45 internal. Flash + console + JTAG = USB-CDC (IO19/20)."
- note added: "the 5 V rail -> ~3 W quieter alarm. Firmware: LEDs+audio <= ~12 W."
- note added: "use MCP internal pull-ups. Encoder A/B -> hardware PCNT (IO47/48)."

Commit message: kicad2, pass 3
Parts:
- J5: footprint Connector_FFC-FPC:Hirose_FH34SRJ-10S-0.5SH_1x10-1MP_P0.50mm_Horizontal -> Connector_FFC-FPC:Hirose_FH12-10S-0.5SH_1x10-1MP_P0.50mm_Horizontal
Connections:
- net +5V: now also C121.1, C122.1, C123.1, C124.1, R40.1, U5.6 (VOUT), U6.1 (EN), U6.4 (VIN)
- net GND: now also D1.2 (A2), D12.2 (A2); no longer D1.1 (A1), D12.1 (A1)
- net PVDD: now also U9.21 (PVDD), U9.28 (PVDD)
- net VBAT: now also D12.1 (A1), U5.3 (VIN), U7.3 (VIN); no longer D12.2 (A2), R22.1
- net VBUS: now also D1.1 (A1); no longer D1.2 (A2)
- net at U11.5 (AO2), U11.6 (AO2): now also J4.2 (Pin_2); no longer J4.1 (Pin_1)
- net at U11.7 (BO2), U11.8 (BO2): now also J4.3 (Pin_3); no longer J4.2 (Pin_2)
- net at U11.11 (BO1), U11.12 (BO1): now also J4.4 (Pin_4); no longer J4.3 (Pin_3)
- net at U12.1 (AO1), U12.2 (AO1): now also J4.5 (Pin_5); no longer J4.4 (Pin_4)
- net at U12.5 (AO2), U12.6 (AO2): now also J4.6 (Pin_6); no longer J4.5 (Pin_5)
- net at U12.7 (BO2), U12.8 (BO2): now also J4.7 (Pin_7); no longer J4.6 (Pin_6)
- net at U12.11 (BO1), U12.12 (BO1): now also J4.8 (Pin_8); no longer J4.7 (Pin_7)
- net at C180.2, C182.2, L5.1: now also U9.20 (SPK_OUTB+), U9.29 (SPK_OUTA+); no longer C182.1, U9.19 (BSTRPB+)
- net at U5.5 (SW): now also L2.2
- net at D20.2 (A), L4.2, U7.2 (SW): now also U7.1 (SW)
- net at BT1.1 (Pin_1), Q2.2 (S), R20.1: now also R22.1
- net at R71.2: now also J6.8 (DAT1); no longer J6.1 (DAT2)
- net at R72.2: now also J6.1 (DAT2); no longer J6.8 (DAT1)
- net at U9.23 (SPK_OUTB-): now also C181.2, C183.2, L6.1, U9.26 (SPK_OUTA-)
- net at U11.1 (AO1), U11.2 (AO1): now also J4.1 (Pin_1)
- new net: C183.1, U9.24 (BSTRPB-)
- new net: C181.1, U9.25 (BSTRPA-)
- new net: C182.1, U9.19 (BSTRPB+)
Other:
- moved on the sheet: D1, D12

Commit message: kicad2, pass 4 (final)
Other:
- note added: "+3V3"
- note added: "HOW TO READ THIS SHEET"
- note added: "I2S, MCPWM, encoder) are drawn as wires; GND / +3V3 / +5V taps"
- note added: "MCU centre, peripherals right. Power paths and MCU buses (SPI,"
- note added: "Off-board parts (display, SD, sensors, speaker, motor, LED"
- note added: "One page, laid out like block_diagram.drawio: power flows left,"
- note added: "and named labels connect by name (same name = same net)."
- note added: "strips, cell) enter through connectors J1..J9 / BT1."

Commit message: kicad2 validation phase
Other:
- note added: "Layout: C220/C221 at the J5 VDDA/VDD pins; C222/C223 at the J6 VDD pin."
- note added: "Layout: each driver's 10uF+100nF go at its VM pins, the 100nF at its VCC pin."
