File: kicad-sensor/sensor.kicad_pcb (KiCad board)
At the start: 4 copper layers, 30 x 16 mm, 33 parts, among them J1 To main board J7, U1 BNO085, U2 BME688, U3 TSL25911FN, Y1 32.768kHz

Commit message: sensor board v0.2: action kicad-sensor/REVIEW.md
Schematic, PCB, generators, QA checks and docs brought into one consistent
state. ERC 0 violations, DRC 0 violations / 0 unconnected / 0 parity issues,
gen/pcb_check.py 33/33, stamp_bom.py idempotent.

Safety and correctness
- #1  Address straps R3/R4/R10/R11 0R -> 10k. Fitting both halves of either
      pair shorted the MAIN board's +3V3 to GND through 0 ohm; it now costs
      330 uA and the part enumerates at a visible wrong address. PCB Value
      fields follow the schematic.
- W1  gen/pcb_build.py refuses to run without PCB_BUILD_WIPE_ROUTING=1. It
      produced the old 2-layer unrouted placement and would wipe the routing.
- #4  The reversed-harness / J10 mis-mate hazard is now a warning block on
      the schematic sheet, in README.md and on J10's own BOM line.

Versioning (#11) - one scheme in three places
- PCB title block added (there was none), schematic rev "A" -> "v0.2", silk
  SENSE v0.1 -> SENSE v0.2. pcb_check.py fails if the three disagree.

PCB (#7 #8 #10 #14)
- Thermal-island copper 21.0 -> 18.2 mm, GND share 8.8 -> 6.0 mm: the GND
  daisy-chain that ran down the inside of the island is replaced by the
  shortest exits that reach the pour.
- C4/C7 +0.175 mm east (all U1's and Y1's courtyards allow), restoring
  requirement 5 "nothing on the back behind U2".
- All five hidden reference designators un-hidden, the four stray free silk
  texts removed; only H1/H2 stay hidden, and that is now asserted.
- U3 moved to a project-local footprint fork,
  sensor:AMS_TSL25911FN_ALSWindow - the stock silk crosses the optical
  window 1.31 mm from the photodiode. Forked, not hand-edited, so Update
  Footprints from Library cannot undo it and DRC stays clean.

QA re-baselined (#6 #9 #15)
- pcb_check.py judged the generated 2-layer placement; four checks failed
  against a board that is fine. Clearance is now judged on pad-to-pad
  copper (>= 0.60 mm everywhere) with the six sub-0.22 mm courtyard pairs
  named a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
Parts:
- R10, R3: value 0R -> 10k
- R11, R4: value 0R (DNP) -> 10k (DNP)
- U3: footprint OptoDevice:AMS_TSL25911FN -> sensor:AMS_TSL25911FN_ALSWindow
- moved C4 0.17 mm to (7.88, 8.90)
- moved C7 0.17 mm to (7.88, 10.7)
Routing:
- net GND: track 42.0 -> 39.0 mm
Other:
- board text added: "SENSE v0.2"
- board text removed: "C11"
- board text removed: "C8"
- board text removed: "R1"
- board text removed: "SENSE v0.1"
- board text removed: "TP1"
- board text removed: "U1"
Changed lines of the file:
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@@
 	)
 	(paper "A4")
+	(title_block
+		(title "Wooden Smart Clock — sensor board")
+		(date "2026-08-07")
+		(rev "v0.2")
+	)
 	(layers
 		(0 "F.Cu" signal)
@@
 		(tags "capacitor")
 		(property "Reference" "C11"
-			(at 0 0 180)
+			(at 0 -1.5 180)
 			(layer "F.SilkS")
-			(hide yes)
 			(effects
 				(font
@@
 			)
 		)
-		(property "Value" "0R"
+		(property "Value" "10k"
 			(at 0 1.43 180)
 			(layer "F.Fab")
@@
 			)
 		)
-		(property "Description" "RES 0 OHM JUMPER 1/10W 0603"
+		(property "Description" "RES 10K OHM 1% 1/10W 0603"
 			(at 0 0 180)
 			(layer "F.Fab")
@@
 			)
 		)
-		(property "MPN" "RC0603JR-070RL"
+		(property "MPN" "RC0603FR-0710KL"
 			(at 0 0 180)
 			(layer "F.Fab")
@@
 			)
 		)
-		(property "Value" "0R (DNP)"
+		(property "Value" "10k (DNP)"
 			(at 0 1.43 0)
 			(layer "F.Fab")
@@
 			)
 		)
-		(property "Description" "RES 0 OHM JUMPER 1/10W 0603"
+		(property "Description" "RES 10K OHM 1% 1/10W 0603"
 			(at 0 0 0)
 			(layer "F.Fab")
@@
 			)
 		)
-		(property "MPN" "RC0603JR-070RL"
+		(property "MPN" "RC0603FR-0710KL"
 			(at 0 0 0)
 			(layer "F.Fab")
@@
 			)
 		)
-		(property "Notes" "DO NOT POPULATE — alternate BME688 address strap — fit INSTEAD OF R10 for 0x76 (both fitted = +3V3 shorted to GND through 0 ohm)"
+		(property "Notes" "DO NOT POPULATE — alternate BME688 address strap — fit INSTEAD OF R10 for 0x76 (both fitted = +3V3 to GND through 20k, 330 uA, wrong address)"
 			(at 0 0 0)
 			(layer "F.Fab")
@@
 		)
 	)
-	(footprint "OptoDevice:AMS_TSL25911FN"
+	(footprint "sensor:AMS_TSL25911FN_ALSWindow"
 		(layer "F.Cu")
 		(at 11.5 3.6)
@@
 		(attr smd)
 		(duplicate_pad_numbers_are_jumpers no)
-		(fp_line
-			(start -1 -1.31)
-			(end 1 -1.31)
-			(stroke
-				(width 0.12)
-				(type solid)
-			)
-			(layer "F.SilkS")
-		)
-		(fp_line
-			(start -1 1.31)
-			(end 1 1.31)
-			(stroke
-				(width 0.12)
-				(type solid)
-			)
-			(layer "F.SilkS")
-		)
 		(fp_poly
 			(pts
-				(xy -1.23 -1.01) (xy -1.51 -1.01) (xy -1.23 -1.29) (xy -1.23 -1.01)
+				(xy -1.46 -1.61) (xy -1.74 -1.61) (xy -1.46 -1.89) (xy -1.46 -1.61)
 			)
 			(stroke
@@
 			)
 		)
-		(property "Value" "0R (DNP)"
+		(property "Value" "10k (DNP)"
 			(at 0 -1.43 0)
 			(layer "B.Fab")
@@
 			)
 		)
-		(property "Description" "RES 0 OHM JUMPER 1/10W 0603"
+		(property "Description" "RES 10K OHM 1% 1/10W 0603"
 			(at 0 0 0)
 			(layer "B.Fab")
@@
 			)
 		)
-		(property "MPN" "RC0603JR-070RL"
+		(property "MPN" "RC0603FR-0710KL"
 			(at 0 0 0)
 			(layer "B.Fab")
@@
 			)
 		)
-		(property "Notes" "DO NOT POPULATE — alternate BNO085 address strap — fit INSTEAD OF R3 for 0x4B (both fitted = +3V3 shorted to GND through 0 ohm)"
+		(property "Notes" "DO NOT POPULATE — alternate BNO085 address strap — fit INSTEAD OF R3 for 0x4B (both fitted = +3V3 to GND through 20k, 330 uA, wrong address)"
 			(at 0 0 0)
 			(layer "B.Fab")
@@
 		(tags "LGA 28 5.2x3.8mm P0.5mm BNO085 BNO080 BNO086 IMU")
 		(property "Reference" "U1"
-			(at 4.38 1.6 180)
+			(at -1 -2.5 180)
 			(layer "B.SilkS")
-			(hide yes)
 			(effects
 				(font
@@
 	(footprint "Capacitor_SMD:C_0603_1608Metric"
 		(layer "B.Cu")
-		(at 7.7 10.7 180)
+		(at 7.875 10.7 180)
 		(descr "Capacitor SMD 0603 (1608 Metric), square (rectangular) end terminal, IPC-7351 nominal, (Body size source: IPC-SM-782 page 76, https://www.pcb-3d.com/wordpress/wp-content/uploads/ipc-sm-782a_amendment_1_and_2.pdf)")
 		(tags "capacitor")
@@
 		(tags "test point SMD pad")
 		(property "Reference" "TP1"
-			(at 2.87 1.6 0)
+			(at 0.1 -1.2 0)
 			(layer "B.SilkS")
-			(hide yes)
 			(effects
 				(font
@@
 	(footprint "Capacitor_SMD:C_0603_1608Metric"
 		(layer "B.Cu")
-		(at 7.7 8.9 180)
+		(at 7.875 8.9 180)
 		(descr "Capacitor SMD 0603 (1608 Metric), square (rectangular) end terminal, IPC-7351 nominal, (Body size source: IPC-SM-782 page 76, https://www.pcb-3d.com/wordpress/wp-content/uploads/ipc-sm-782a_amendment_1_and_2.pdf)")
 		(tags "capacitor")
@@
 		(tags "capacitor")
 		(property "Reference" "C8"
-			(at -4.485 2.4 180)
+			(at 2.275 -0.2 180)
 			(layer "B.SilkS")
-			(hide yes)
 			(effects
 				(font
@@
 			)
 		)
-		(property "Package" "JST ZH 1.50mm 6-pos TH vertical"
+		(property "Package" "JST ZH 1.50mm 6-pos TH vertical, 2.7mm tail"
 			(at 0 0 0)
 			(layer "B.Fab")
@@
 			)
 		)
-		(property "Notes" "Mates main-board J7 1:1 over the 6-way ZH harness (same part both ends). The only through-hole part on this board — hand-solder it after reflow, or have it fitted as a second operation"
+		(property "Notes" "DigiKey 455-B6B-ZR-ND — $0.24, Active, 9,478 pcs (2026-08-07). Mates main-board J7 1:1 over the 6-way ZH harness (same part both ends); ZHR-6 housing + A06ZR pre-crimped cable. JST specs the 3.4 mm tail (B6B-ZR-3.4) for 1.6 mm board thickness, but that variant is made-to-order only (MOQ 2,000, 16 wk) — 2.7 mm leaves 1.1 mm protruding here, which solders fine; deviation accepted, see ../PCB_NOTES.md. The only through-hole part on this board — hand-solder it after reflow, or have it fitted as a third operation"
 			(at 0 0 0)
 			(layer "B.Fab")
@@
 			)
 		)
-		(property "Value" "0R"
+		(property "Value" "10k"
 			(at 0 -1.43 0)
 			(layer "B.Fab")
@@
 			)
 		)
-		(property "Description" "RES 0 OHM JUMPER 1/10W 0603"
+		(property "Description" "RES 10K OHM 1% 1/10W 0603"
 			(at 0 0 0)
 			(layer "B.Fab")
@@
 			)
 		)
-		(property "MPN" "RC0603JR-070RL"
+		(property "MPN" "RC0603FR-0710KL"
 			(at 0 0 0)
 			(layer "B.Fab")
@@
 		(tags "resistor")
 		(property "Reference" "R1"
-			(at -2.1 0 90)
+			(at 1.9 0.5 90)
 			(layer "B.SilkS")
-			(hide yes)
 			(effects
 				(font
@@
 		)
 	)
-	(gr_text "C11"
-		(at 3 15 0)
-		(layer "F.SilkS")
-		(effects
-			(font
-				(size 0.8 0.8)
-				(thickness 0.12)
-			)
-		)
-	)
 	(gr_text "ENVIR"
 		(at 4.5 6.4 0)
@@
 	)
 	(gr_text "ALS"
-		(at 12 1.5 0)
+		(at 11.5 6.3 0)
 		(layer "F.SilkS")
 		(effects
@@
 		)
 	)
-	(gr_text "SENSE v0.1"
+	(gr_text "SENSE v0.2"
 		(at 24.5 2.5 0)
 		(layer "F.SilkS")
@@
 		)
 	)
-	(gr_text "TP1"
-		(at 15.5 1.5 0)
-		(layer "B.SilkS")
-		(effects
-			(font
-				(size 0.8 0.8)
-				(thickness 0.12)
-			)
-			(justify left bottom mirror)
-		)
-	)
-	(gr_text "U1"
-		(at 11.5 4.5 0)
-		(layer "B.SilkS")
-		(effects
-			(font
-				(size 0.8 0.8)
-				(thickness 0.12)
-			)
-			(justify mirror)
-		)
-	)
-	(gr_text "C8"
-		(at 18.5 10.5 0)
-		(layer "B.SilkS")
-		(effects
-			(font
-				(size 0.8 0.8)
-				(thickness 0.12)
-			)
-			(justify mirror)
-		)
-	)
-	(gr_text "R1"
-		(at 20.5 11 90)
-		(layer "B.SilkS")
-		(effects
-			(font
-				(size 0.8 0.8)
-				(thickness 0.12)
-			)
-			(justify mirror)
-		)
-	)
 	(gr_text "VENT"
 		(at 4.5 6.7 0)
@@
 	)
 	(segment
-		(start 8.8217 9.2467)
-		(end 10.75 9.2467)
+		(start 8.997 9.247)
+		(end 10.75 9.247)
 		(width 0.25)
 		(layer "B.Cu")
@@
 	)
 	(segment
-		(start 8.475 8.9)
-		(end 8.8217 9.2467)
+		(start 8.65 8.9)
+		(end 8.997 9.247)
 		(width 0.25)
 		(layer "B.Cu")
@@
 	)
 	(segment
-		(start 8.475 8.9)
-		(end 8.475 7.25)
+		(start 8.65 8.9)
+		(end 8.65 7.25)
 		(width 0.25)
 		(layer "B.Cu")
@@
 	)
 	(segment
-		(start 6.925 11.425)
-		(end 8 12.5)
-		(width 0.25)
-		(layer "B.Cu")
-		(net "GND")
-	)
-	(segment
-		(start 6.925 8.9)
-		(end 6.925 10.7)
-		(width 0.25)
-		(layer "B.Cu")
-		(net "GND")
-	)
-	(segment
 		(start 10.75 6.25)
 		(end 11 6.5)
@@
 	)
 	(segment
-		(start 6.925 7.1)
-		(end 6.925 8.9)
+		(start 7.1 7.275)
+		(end 6.925 7.1)
 		(width 0.25)
 		(layer "B.Cu")
@@
 	)
 	(segment
-		(start 6.925 10.7)
-		(end 6.925 11.425)
+		(start 12.25 7.75)
+		(end 13 7)
 		(width 0.25)
 		(layer "B.Cu")
@@
 	)
 	(segment
-		(start 12.25 7.75)
-		(end 13 7)
+		(start 7.1 8.9)
+		(end 7.1 7.275)
 		(width 0.25)
 		(layer "B.Cu")
@@
 	)
 	(segment
+		(start 7.1 10.7)
+		(end 7.8 11.4)
+		(width 0.25)
+		(layer "B.Cu")
+		(net "GND")
+	)
+	(segment
 		(start 10.25 6.1875)
 		(end 10.1875 6.25)
@@
 	)
 	(segment
-		(start 8.475 10.7)
+		(start 8.65 10.7)
 		(end 10.75 10.7)
 		(width 0.25)
