File: kicad-sensor/sensor.kicad_sch (KiCad schematic)
At the start: 31 parts, among them J1 To main board J7, U1 BNO085, U2 BME688, U3 TSL25911FN, Y1 32.768kHz

Commit message: correct BOM options
Parts:
- C1: MPN (none) -> CL21A106KAYNNNE; Manufacturer (none) -> Samsung Electro-Mechanics; Notes (none) -> Substitution OK - same value/tolerance/voltage/dielectric/s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; Package (none) -> 0805
- C10, C11, C2, C3, C4, C6, C9: MPN (none) -> CL10B104KB8NNNC; Manufacturer (none) -> Samsung Electro-Mechanics; Notes (none) -> Substitution OK - same value/tolerance/voltage/dielectric/s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; Package (none) -> 0603
- C12, C5: MPN (none) -> CL10B105KA8NNNC; Manufacturer (none) -> Samsung Electro-Mechanics; Notes (none) -> Substitution OK - same value/tolerance/voltage/dielectric/s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; Package (none) -> 0603
- C7, C8: MPN (none) -> CL10C220JB8NNNC; Manufacturer (none) -> Samsung Electro-Mechanics; Notes (none) -> Substitution OK - same value/tolerance/voltage/dielectric/s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; Package (none) -> 0603
- J1: MPN (none) -> B6B-ZR(LF)(SN); Manufacturer (none) -> JST Sales America; Notes (none) -> Mates main-board J7 1:1 over the 6-way ZH harness (same par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; Package (none) -> JST ZH 1.50mm 6-pos TH vertical
- R1, R12, R2, R5, R6, R7, R8, R9: MPN (none) -> RC0603FR-0710KL; Manufacturer (none) -> YAGEO; Notes (none) -> Substitution OK - same value/tolerance/voltage/dielectric/s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; Package (none) -> 0603
- R10, R3: MPN (none) -> RC0603JR-070RL; Manufacturer (none) -> YAGEO; Notes (none) -> Substitution OK - same value/tolerance/voltage/dielectric/s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; Package (none) -> 0603
- R11: MPN (none) -> RC0603JR-070RL; Manufacturer (none) -> YAGEO; Notes (none) -> DO NOT POPULATE — alternate BME688 address strap — fit INST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; Package (none) -> 0603; now not fitted
- R4: MPN (none) -> RC0603JR-070RL; Manufacturer (none) -> YAGEO; Notes (none) -> DO NOT POPULATE — alternate BNO085 address strap — fit INST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; Package (none) -> 0603; now not fitted
- TP1, TP2: now left out of the parts list
- U1: MPN (none) -> BNO085; Manufacturer (none) -> CEVA Technologies; Notes (none) -> DigiKey 1888-1006-1-ND (cut tape) — $13.57, Active, 324 pcs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; Package (none) -> LGA-28 5.2x3.8x1.1mm, 0.5mm pitch
- U2: MPN (none) -> BME688; Manufacturer (none) -> Bosch Sensortec; Notes (none) -> DigiKey 828-BME688CT-ND — $8.99 single, Active, 9.3k pcs (2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; Package (none) -> LGA-8 3.0x3.0x0.93mm
- U3: MPN (none) -> TSL25911FN; Manufacturer (none) -> ams-OSRAM; Notes (none) -> DigiKey TSL25911FNTR-ND (product 4162547) — $1.74, Active, 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; Package (none) -> WFDFN-6 2.0x2.0mm
- Y1: MPN (none) -> ABS07-32.768KHZ-T; Manufacturer (none) -> Abracon; Notes (none) -> Same part as the main board's RTC crystal — one line covers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; Package (none) -> SMD 3.2x1.5mm 2-pin
