File: kicad-sensor/sensor.kicad_sch (KiCad schematic)
At the start: 31 parts, among them J1 To main board J7, U1 BNO085, U2 BME688, U3 TSL25911FN, Y1 32.768kHz

Commit message: sensor board v0.2: action kicad-sensor/REVIEW.md
Schematic, PCB, generators, QA checks and docs brought into one consistent
state. ERC 0 violations, DRC 0 violations / 0 unconnected / 0 parity issues,
gen/pcb_check.py 33/33, stamp_bom.py idempotent.

Safety and correctness
- #1  Address straps R3/R4/R10/R11 0R -> 10k. Fitting both halves of either
      pair shorted the MAIN board's +3V3 to GND through 0 ohm; it now costs
      330 uA and the part enumerates at a visible wrong address. PCB Value
      fields follow the schematic.
- W1  gen/pcb_build.py refuses to run without PCB_BUILD_WIPE_ROUTING=1. It
      produced the old 2-layer unrouted placement and would wipe the routing.
- #4  The reversed-harness / J10 mis-mate hazard is now a warning block on
      the schematic sheet, in README.md and on J10's own BOM line.

Versioning (#11) - one scheme in three places
- PCB title block added (there was none), schematic rev "A" -> "v0.2", silk
  SENSE v0.1 -> SENSE v0.2. pcb_check.py fails if the three disagree.

PCB (#7 #8 #10 #14)
- Thermal-island copper 21.0 -> 18.2 mm, GND share 8.8 -> 6.0 mm: the GND
  daisy-chain that ran down the inside of the island is replaced by the
  shortest exits that reach the pour.
- C4/C7 +0.175 mm east (all U1's and Y1's courtyards allow), restoring
  requirement 5 "nothing on the back behind U2".
- All five hidden reference designators un-hidden, the four stray free silk
  texts removed; only H1/H2 stay hidden, and that is now asserted.
- U3 moved to a project-local footprint fork,
  sensor:AMS_TSL25911FN_ALSWindow - the stock silk crosses the optical
  window 1.31 mm from the photodiode. Forked, not hand-edited, so Update
  Footprints from Library cannot undo it and DRC stays clean.

QA re-baselined (#6 #9 #15)
- pcb_check.py judged the generated 2-layer placement; four checks failed
  against a board that is fine. Clearance is now judged on pad-to-pad
  copper (>= 0.60 mm everywhere) with the six sub-0.22 mm courtyard pairs
  named a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
Parts:
- J1: Notes Mates main-board J7 1:1 over the 6-way ZH harness (same par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 -> DigiKey 455-B6B-ZR-ND — $0.24, Active, 9,478 pcs (2026-08-0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; Package JST ZH 1.50mm 6-pos TH vertical -> JST ZH 1.50mm 6-pos TH vertical, 2.7mm tail
- R10, R3: value 0R -> 10k; MPN RC0603JR-070RL -> RC0603FR-0710KL
- R11: value 0R (DNP) -> 10k (DNP); MPN RC0603JR-070RL -> RC0603FR-0710KL; Notes DO NOT POPULATE — alternate BME688 address strap — fit INSTEAD OF R10 for 0x76 (both fitted = +3V3 shorted to GND through 0 ohm) -> DO NOT POPULATE — alternate BME688 address strap — fit INSTEAD OF R10 for 0x76 (both fitted = +3V3 to GND through 20k, 330 uA, wrong address)
- R4: value 0R (DNP) -> 10k (DNP); MPN RC0603JR-070RL -> RC0603FR-0710KL; Notes DO NOT POPULATE — alternate BNO085 address strap — fit INSTEAD OF R3 for 0x4B (both fitted = +3V3 shorted to GND through 0 ohm) -> DO NOT POPULATE — alternate BNO085 address strap — fit INSTEAD OF R3 for 0x4B (both fitted = +3V3 to GND through 20k, 330 uA, wrong address)
- U3: footprint OptoDevice:AMS_TSL25911FN -> sensor:AMS_TSL25911FN_ALSWindow
Other:
- note added: "(GPPU.3 = 1) so that pin does not float when this board is unplugged. See FIRMWARE.md §6.5."
- note added: "+ 0.3 V at any logic pin", series-limited only by the main board's R97 10k: assume U1 is destroyed."
- note added: "16 wk), and 2.7 mm leaves 1.1 mm protruding, which solders fine. Deviation accepted 2026-08-07."
- note added: "5 V on +3V3 and takes all three sensors at once. Label both cables; check before first power-up."
- note added: "Address straps are 10k, not 0R: R3+R4 or R10+R11 fitted TOGETHER would otherwise short the main"
- note added: "Both ends are ZHR-6 and J1 mirrors J7 1:1, so a cable loaded BACKWARDS plugs in perfectly — and"
- note added: "Bus pull-ups: 4.7k on the main board + R1/R2 10k here ~= 3.2k effective."
- note added: "HARNESS POLARITY IS A DESTRUCTIVE FAULT"
- note added: "Harness must be 1:1 (pin n <-> pin n), NOT reversed — see below."
- note added: "J1 is the ONLY through-hole part: it needs a third operation (selective/hand solder) after both"
- note added: "J1.5 then receives J7.2 +3V3 while this board's VDDIO is 0 V. BNO08X abs max (Fig. 6-1) is "VDDIO"
- note added: "J10 (knob) is the SAME ZH 1x06 header 13.5 mm from J7, with +5 V on pin 2 — that mis-mate puts"
- note added: "NO aqueous wash, no flux over the port, no conformal coat, no silicone/siloxane exposure. Bosch's"
- note added: "Rules are Bosch's HSMI, which §7.7 defers to: ../datasheet/sensor_env_bme68x_hsmi.pdf (no BME688-"
- note added: "Tail: JST specs the 3.4 mm variant for a 1.6 mm board, but B6B-ZR-3.4 is made-to-order (MOQ 2000,"
- note added: "U2 HANDLING (BME688) A metal-oxide gas hotplate does not fail when mishandled, it reads a wrong VOC"
- note added: "and only here — it lands on main-board MCP23017 GPB3, which must enable its internal pull-up"
- note added: "baseline forever. MSL 1 (no bake), peak reflow 260 C (§7.6), and >= 50 um solder height AFTER"
- note added: "board's +3V3 to GND. Fit exactly one of each pair; the alternates are flagged DNP."
- note added: "harness (B6B-ZR both ends, 1:1). +3V3 and GND arrive on the cable; there is no regulator here."
- note added: "reflow (§7.7, for mechanical decoupling) — that is a stencil-thickness decision, not a layout one."
- note added: "reflows — price that before committing, it is usually quoted per board, not per joint."
- note added: "specific HSMI is published; the BME680 one is the same package, lid vent and MOX element)."
- note added: "when the harness is unplugged). J7.6 ALS_INT = TSL2591 INT, open drain, pulled up by R12 HERE"
- note removed: "BEFORE FAB Check the stock LGA-28 land (generic IPC pattern) against BNO08X datasheet Fig. 7-2:"
- note removed: "Harness must be 1:1 (pin n <-> pin n), NOT reversed."
- note removed: "Pull-ups: 4.7k on the main board + R1/R2 10k here ~= 3.2k effective."
- note removed: "harness (B6B-ZR both ends, 1:1). Rails: +3V3 and GND arrive on the cable; no regulator here."
- note removed: "its pads sit ~0.10-0.13 mm further out than CEVA's drawing. Numbering/arrangement do match."
- note removed: "the main board leaves that pin unconnected today, so it is a wire-in-place-for-later."
- note removed: "when the harness is unplugged). J7.6 ALS_INT = TSL2591 INT, open drain, pulled up by R12 here —"

Commit message: BME688 handling into the BOM line; close the 3 vendor-drawing checks
Sensor board — the handling rules now ship with the BOM
U2's Notes field carries the full Bosch HSMI contract: MSL 1, 260 C for
20-40 s, max 3 reflow cycles, minimum 50 um solder height after reflow, no
aqueous wash, vent covered for any cleaning step, no siloxanes anywhere
near it, and the reason it matters - a washed or siloxane-exposed hotplate
does not fail electrically, it reads a wrong VOC baseline for ever, so
nothing at incoming test will catch it.

It goes in Notes specifically so it travels with the exported CSV to the
assembly house, rather than living in a README they will never open. The
same text is stamped into both sensor.kicad_sch and sensor.kicad_pcb, so
the kicad-cli BOM and the PCBWay plug-in BOM both carry it. Verified by
exporting the CSV: 12 lines, U2's note 1116 chars, rules present.

Main board — the three "scraps a board" items are closed
The board owner validated all three custom footprints against their vendor
drawings on 2026-08-08:
- Juken X40-879 (#25): peg holes and shaft hole confirmed. AN-JST-001 is no
  longer a fab gate. It stays the only source for insertion force and peg
  length vs board thickness, so the 2.0 mm-stackup discussion re-opens it -
  noted in place rather than deleted.
- Keystone 1043: pegs, index post and PC-pin span confirmed. The footprint's
  own "VERIFY vs the Keystone 1043 drawing before fab" descr note is
  replaced with the verification, so the file no longer contradicts the
  review.
- GCT USB4160 USB-C land: confirmed.

That clears the whole class the pre-fab audit called "the ones that scrap a
whole board rather than cost a bodge wire". What remains before ordering is
recorded there: two stock checks (R1 RC1206FR-071KL, C172 EEH-ZA1E101P)
which gate assembly rather than bare-board fab, and the fact that neither
project has exported Gerbers or been through a fab's DFM.

Verification unchanged: sensor ERC 0 / DRC 0 / pcb_check 33/33; main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
Parts:
- U2: Notes DigiKey 828-BME688CT-ND — $8.99 single, Active, 9.3k pcs (2026-08-01; datasheet/README.md §12's ~$5 is the 3k reel price). Gas sensor: do not conformal-coat, keep the vent clear -> DigiKey 828-BME688CT-ND — $8.99 single, Active, 9.3k pcs (2026-08-01; datasheet/README.md §12's ~$5 is the 3k reel price). *** HANDLING IS CONTRACTUAL — GAS SENSOR, SEE BOSCH HSMI (BST-BME680-HS000-06, supplied with this package). (1) MSL 1, no bake. (2) Peak reflow 260 C for 20-40 s, MAX 3 REFLOW CYCLES — this board is double-sided, so U2 already sees two. (3) MINIMUM 50 um SOLDER HEIGHT AFTER REFLOW — this is a stencil thickness decision and must be confirmed BEFORE the run; it is what mechanically decouples the die from the board. (4) NO AQUEOUS WASH and no flux over the vent hole; if any cleaning step is used the vent must first be covered with a silicone-free protective layer. No-clean process preferred. (5) NO SILICONE / SILOXANE ANYWHERE NEAR THIS PART — gloves, adhesives, coatings, packaging. Permanent VOC poisoning. (6) No conformal coat, no underfill, no ultrasonic welding, nothing sharp in the vent, no rear-side handling. A part that has been washed, fluxed over or siloxane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
Changed lines of the file:
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@@
 			)
 		)
-		(property "Notes" "DigiKey 828-BME688CT-ND — $8.99 single, Active, 9.3k pcs (2026-08-01; datasheet/README.md §12's ~$5 is the 3k reel price). Gas sensor: do not conformal-coat, keep the vent clear"
+		(property "Notes" "DigiKey 828-BME688CT-ND — $8.99 single, Active, 9.3k pcs (2026-08-01; datasheet/README.md §12's ~$5 is the 3k reel price). *** HANDLING IS CONTRACTUAL — GAS SENSOR, SEE BOSCH HSMI (BST-BME680-HS000-06, supplied with this package). (1) MSL 1, no bake. (2) Peak reflow 260 C for 20-40 s, MAX 3 REFLOW CYCLES — this board is double-sided, so U2 already sees two. (3) MINIMUM 50 um SOLDER HEIGHT AFTER REFLOW — this is a stencil thickness decision and must be confirmed BEFORE the run; it is what mechanically decouples the die from the board. (4) NO AQUEOUS WASH and no flux over the vent hole; if any cleaning step is used the vent must first be covered with a silicone-free protective layer. No-clean process preferred. (5) NO SILICONE / SILOXANE ANYWHERE NEAR THIS PART — gloves, adhesives, coatings, packaging. Permanent VOC poisoning. (6) No conformal coat, no underfill, no ultrasonic welding, nothing sharp in the vent, no rear-side handling. A part that has been washed, fluxed over or siloxane-exposed does NOT fail electrically — it reads a wrong gas baseline for ever, so incoming test will not catch it. ***"
 			(at 76.2 153.67 0)
 			(hide yes)
